Commit message: Add ros2_control and gripper inertial settings

File: ros2_ws/src/robot_arm_description/urdf/robot_arm.urdf (robot description, URDF)
Before this commit: robot robot_arm, 10 links, 9 joints
Links:
- link gripper_base: mass None -> 0.1
- link left_finger: mass None -> 0.05
- link right_finger: mass None -> 0.05

Commit message: fix: restore gripper URDF with MoveIt config

File: ros2_ws/src/robot_arm_description/urdf/robot_arm.urdf (robot description, URDF)
Before this commit: robot robot_arm, 10 links, 9 joints
Links:
- link gripper_base: mass 0.1 -> None
- link left_finger: mass 0.05 -> None
- link right_finger: mass 0.05 -> None

Commit message: fix(urdf):1차수정버전교체
urdf몸체만 있는 버전으로 수정한 뒤 업로드, 그리퍼 모듈화 구조를 위한 소프트웨어 작동 방식 고려 필요

File: ros2_ws/src/robot_arm_description/urdf/robot_arm.urdf (robot description, URDF)
Before this commit: robot robot_arm, 10 links, 9 joints
Links:
- removed link gripper_base
- removed link left_finger
- removed link link_1
- removed link link_2
- removed link link_3
- removed link link_4
- removed link link_5
- removed link link_6
- removed link right_finger
- added link Adapter_A_1, mass 0.09838512042156757; collision mesh filename=package://robot_arm_description/meshes/Adapter_A_1.stl scale=0.001 0.001 0.001; visual mesh filename=package://robot_arm_description/meshes/Adapter_A_1.stl scale=0.001 0.001 0.001
- added link Adapter_A_1_1, mass 0.09838512042156751; collision mesh filename=package://robot_arm_description/meshes/Adapter_A_1_1.stl scale=0.001 0.001 0.001; visual mesh filename=package://robot_arm_description/meshes/Adapter_A_1_1.stl scale=0.001 0.001 0.001
- added link Adapter_B_1, mass 0.0383693503096125; collision mesh filename=package://robot_arm_description/meshes/Adapter_B_1.stl scale=0.001 0.001 0.001; visual mesh filename=package://robot_arm_description/meshes/Adapter_B_1.stl scale=0.001 0.001 0.001
- added link Adapter_B_1_1_1, mass 0.0836288961017048; collision mesh filename=package://robot_arm_description/meshes/Adapter_B_1_1_1.stl scale=0.001 0.001 0.001; visual mesh filename=package://robot_arm_description/meshes/Adapter_B_1_1_1.stl scale=0.001 0.001 0.001
- added link Adapter_b_1_1, mass 0.1507674746734739; collision mesh filename=package://robot_arm_description/meshes/Adapter_b_1_1.stl scale=0.001 0.001 0.001; visual mesh filename=package://robot_arm_description/meshes/Adapter_b_1_1.stl scale=0.001 0.001 0.001
- added link Bottom_Cylinder_1, mass 2.7522236601038736; collision mesh filename=package://robot_arm_description/meshes/Bottom_Cylinder_1.stl scale=0.001 0.001 0.001; visual mesh filename=package://robot_arm_description/meshes/Bottom_Cylinder_1.stl scale=0.001 0.001 0.001
- added link Bottom_top_1, mass 0.7527923586440036; collision mesh filename=package://robot_arm_description/meshes/Bottom_top_1.stl scale=0.001 0.001 0.001; visual mesh filename=package://robot_arm_description/meshes/Bottom_top_1.stl scale=0.001 0.001 0.001
- added link GearBox1_1, mass 2.039024001006148; collision mesh filename=package://robot_arm_description/meshes/GearBox1_1.stl scale=0.001 0.001 0.001; visual mesh filename=package://robot_arm_description/meshes/GearBox1_1.stl scale=0.001 0.001 0.001
- added link GearBox2_1, mass 2.0338757908094958; collision mesh filename=package://robot_arm_description/meshes/GearBox2_1.stl scale=0.001 0.001 0.001; visual mesh filename=package://robot_arm_description/meshes/GearBox2_1.stl scale=0.001 0.001 0.001
- added link Link1_1, mass 0.44759500853450696; collision mesh filename=package://robot_arm_description/meshes/Link1_1.stl scale=0.001 0.001 0.001; visual mesh filename=package://robot_arm_description/meshes/Link1_1.stl scale=0.001 0.001 0.001
- added link Link1_1_1, mass 0.40614905152898423; collision mesh filename=package://robot_arm_description/meshes/Link1_1_1.stl scale=0.001 0.001 0.001; visual mesh filename=package://robot_arm_description/meshes/Link1_1_1.stl scale=0.001 0.001 0.001
- added link Link2Bridge2_1, mass 0.6239106311231684; collision mesh filename=package://robot_arm_description/meshes/Link2Bridge2_1.stl scale=0.001 0.001 0.001; visual mesh filename=package://robot_arm_description/meshes/Link2Bridge2_1.stl scale=0.001 0.001 0.001
- added link Link2Bridge_1, mass 0.45400523112316815; collision mesh filename=package://robot_arm_description/meshes/Link2Bridge_1.stl scale=0.001 0.001 0.001; visual mesh filename=package://robot_arm_description/meshes/Link2Bridge_1.stl scale=0.001 0.001 0.001
- added link Link2_1, mass 1.217857292535348; collision mesh filename=package://robot_arm_description/meshes/Link2_1.stl scale=0.001 0.001 0.001; visual mesh filename=package://robot_arm_description/meshes/Link2_1.stl scale=0.001 0.001 0.001
- added link Link2_1_1, mass 1.157660785545272; collision mesh filename=package://robot_arm_description/meshes/Link2_1_1.stl scale=0.001 0.001 0.001; visual mesh filename=package://robot_arm_description/meshes/Link2_1_1.stl scale=0.001 0.001 0.001
- added link Link3Bridge2_1, mass 0.44527262875074014; collision mesh filename=package://robot_arm_description/meshes/Link3Bridge2_1.stl scale=0.001 0.001 0.001; visual mesh filename=package://robot_arm_description/meshes/Link3Bridge2_1.stl scale=0.001 0.001 0.001
- added link Link3Bridge_1, mass 0.6617159687507393; collision mesh filename=package://robot_arm_description/meshes/Link3Bridge_1.stl scale=0.001 0.001 0.001; visual mesh filename=package://robot_arm_description/meshes/Link3Bridge_1.stl scale=0.001 0.001 0.001
- added link Link3_1, mass 0.8074135897799332; collision mesh filename=package://robot_arm_description/meshes/Link3_1.stl scale=0.001 0.001 0.001; visual mesh filename=package://robot_arm_description/meshes/Link3_1.stl scale=0.001 0.001 0.001
- added link Link3_1_1, mass 0.8226070917771181; collision mesh filename=package://robot_arm_description/meshes/Link3_1_1.stl scale=0.001 0.001 0.001; visual mesh filename=package://robot_arm_description/meshes/Link3_1_1.stl scale=0.001 0.001 0.001
- added link Link4_1, mass 0.21556100000000022; collision mesh filename=package://robot_arm_description/meshes/Link4_1.stl scale=0.001 0.001 0.001; visual mesh filename=package://robot_arm_description/meshes/Link4_1.stl scale=0.001 0.001 0.001
- added link Link4_1_1, mass 0.21556100000000022; collision mesh filename=package://robot_arm_description/meshes/Link4_1_1.stl scale=0.001 0.001 0.001; visual mesh filename=package://robot_arm_description/meshes/Link4_1_1.stl scale=0.001 0.001 0.001
- added link Link5_1_1, mass 0.29320833347967973; collision mesh filename=package://robot_arm_description/meshes/Link5_1_1.stl scale=0.001 0.001 0.001; visual mesh filename=package://robot_arm_description/meshes/Link5_1_1.stl scale=0.001 0.001 0.001
- added link Link_5_1, mass 0.3236352008265773; collision mesh filename=package://robot_arm_description/meshes/Link_5_1.stl scale=0.001 0.001 0.001; visual mesh filename=package://robot_arm_description/meshes/Link_5_1.stl scale=0.001 0.001 0.001
- added link Motor0_1, mass 0.664027798614862; collision mesh filename=package://robot_arm_description/meshes/Motor0_1.stl scale=0.001 0.001 0.001; visual mesh filename=package://robot_arm_description/meshes/Motor0_1.stl scale=0.001 0.001 0.001
- added link Motor1_1, mass 0.6640277986148614; collision mesh filename=package://robot_arm_description/meshes/Motor1_1.stl scale=0.001 0.001 0.001; visual mesh filename=package://robot_arm_description/meshes/Motor1_1.stl scale=0.001 0.001 0.001
- added link Motor2_1, mass 0.6640277986148616; collision mesh filename=package://robot_arm_description/meshes/Motor2_1.stl scale=0.001 0.001 0.001; visual mesh filename=package://robot_arm_description/meshes/Motor2_1.stl scale=0.001 0.001 0.001
- added link Motor_1, mass 0.6640277986148609; collision mesh filename=package://robot_arm_description/meshes/Motor_1.stl scale=0.001 0.001 0.001; visual mesh filename=package://robot_arm_description/meshes/Motor_1.stl scale=0.001 0.001 0.001
- added link Plug_1, mass 0.1272431550006768; collision mesh filename=package://robot_arm_description/meshes/Plug_1.stl scale=0.001 0.001 0.001; visual mesh filename=package://robot_arm_description/meshes/Plug_1.stl scale=0.001 0.001 0.001
- added link _Plug2_1, mass 0.12724315500067693; collision mesh filename=package://robot_arm_description/meshes/_Plug2_1.stl scale=0.001 0.001 0.001; visual mesh filename=package://robot_arm_description/meshes/_Plug2_1.stl scale=0.001 0.001 0.001
- link base_link: mass 1.0 -> 0.7385873333015308; geometry collision mesh filename=package://robot_arm_description/meshes/base_link.stl scale=0.001 0.001 0.001; visual mesh filename=package://robot_arm_description/meshes/base_link.stl scale=0.001 0.001 0.001
Joints:
- removed joint gripper_mount
- removed joint joint_4
- removed joint joint_5
- removed joint joint_6
- removed joint left_finger_joint
- removed joint right_finger_joint
- added joint Rigid 21: type fixed, parent base_link, child Bottom_Cylinder_1, origin xyz=0.0 0.01 -0.0005 rpy=0 0 0
- added joint Rigid 22: type fixed, parent Bottom_top_1, child Link1_1, origin xyz=0.0 0.0 0.004 rpy=0 0 0
- added joint Rigid 23: type fixed, parent Bottom_top_1, child Link1_1_1, origin xyz=0.0 0.0 0.004 rpy=0 0 0
- added joint Rigid 42: type fixed, parent Link1_1, child Adapter_B_1, origin xyz=0.06615 -0.001627 0.06 rpy=0 0 0
- added joint Rigid 43: type fixed, parent Adapter_B_1, child Motor_1, origin xyz=-0.0025 -0.004186 0.0 rpy=0 0 0
- added joint Rigid 45: type fixed, parent Adapter_A_1, child GearBox1_1, origin xyz=-0.0093 0.004186 0.0 rpy=0 0 0
- added joint Rigid 46: type fixed, parent GearBox1_1, child Plug_1, origin xyz=-0.1045 -0.004186 0.0 rpy=0 0 0
- added joint Rigid 47: type fixed, parent Plug_1, child Link2_1_1, origin xyz=0.0165 0.0 0.0 rpy=0 0 0
- added joint Rigid 48: type fixed, parent Link2_1_1, child Link2Bridge_1, origin xyz=0.0 0.148151 0.046 rpy=0 0 0
- added joint Rigid 49: type fixed, parent Link2Bridge_1, child Link2_1, origin xyz=0.1626 0.0 0.0 rpy=0 0 0
- added joint Rigid 5: type fixed, parent base_link, child Motor0_1, origin xyz=0.0 0.01 -0.0045 rpy=0 0 0
- added joint Rigid 50: type fixed, parent Link2_1, child Link2Bridge2_1, origin xyz=0.0 0.0175 -0.092 rpy=0 0 0
- added joint Rigid 51: type fixed, parent Link2_1, child Adapter_b_1_1, origin xyz=-0.004 0.144849 0.014 rpy=0 0 0
- added joint Rigid 52: type fixed, parent Adapter_b_1_1, child Motor1_1, origin xyz=-0.0288 0.0 0.0 rpy=0 0 0
- added joint Rigid 54: type fixed, parent Adapter_A_1_1, child GearBox2_1, origin xyz=-0.0093 0.004186 0.0 rpy=0 0 0
- added joint Rigid 55: type fixed, parent GearBox2_1, child _Plug2_1, origin xyz=-0.1045 -0.004186 0.0 rpy=0 0 0
- added joint Rigid 56: type fixed, parent _Plug2_1, child Link3_1, origin xyz=0.0165 0.0 0.0 rpy=0 0 0
- added joint Rigid 57: type fixed, parent Link3_1, child Link3Bridge_1, origin xyz=0.0 -0.10674 0.106 rpy=0 0 0
- added joint Rigid 58: type fixed, parent Link3Bridge_1, child Link3_1_1, origin xyz=0.1943 0.0 0.0 rpy=0 0 0
- added joint Rigid 59: type fixed, parent Link3_1_1, child Link3Bridge2_1, origin xyz=0.0 0.0 -0.092 rpy=0 0 0
- added joint Rigid 60: type fixed, parent Link3_1, child Link4_1, origin xyz=0.0 -0.194627 0.06 rpy=0 0 0
- added joint Rigid 61: type fixed, parent Link4_1, child Link_5_1, origin xyz=0.06865 0.0 0.0 rpy=0 0 0
- added joint Rigid 62: type fixed, parent Link_5_1, child Motor2_1, origin xyz=0.004 -0.063373 0.0 rpy=0 0 0
- added joint Rigid 63: type fixed, parent Motor2_1, child Adapter_B_1_1_1, origin xyz=0.0455 0.0 0.0 rpy=0 0 0
- added joint Rigid 64: type fixed, parent Adapter_B_1_1_1, child Link5_1_1, origin xyz=0.0074 0.004186 0.0 rpy=0 0 0
- added joint Rigid 65: type fixed, parent Link5_1_1, child Link4_1_1, origin xyz=0.0 0.059187 0.0 rpy=0 0 0
- joint joint_1: axis 0 0 1 -> 0.0 0.0 1.0; child link_1 -> Bottom_top_1; limit lower=-3.14 upper=3.14 effort=10 velocity=1.0 -> (none); origin xyz=0 0 0.025 rpy=0 0 0 -> xyz=0.0 0.0 0.0505 rpy=0 0 0; parent base_link -> Motor0_1; type revolute -> continuous
- joint joint_2: axis 0 1 0 -> -1.0 -0.0 0.0; child link_2 -> Adapter_A_1; limit lower=-1.57 upper=1.57 effort=10 velocity=1.0 -> lower=-3.141593 upper=0.0 effort=100 velocity=100; origin xyz=0 0 0.1 rpy=0 0 0 -> xyz=-0.048 0.0 0.0 rpy=0 0 0; parent link_1 -> Motor_1
- joint joint_3: axis 0 1 0 -> -1.0 0.0 0.0; child link_3 -> Adapter_A_1_1; limit lower=-1.57 upper=1.57 effort=10 velocity=1.0 -> lower=0.0 upper=3.665191 effort=100 velocity=100; origin xyz=0 0 0.2 rpy=0 0 0 -> xyz=-0.048 0.0 0.0 rpy=0 0 0; parent link_2 -> Motor1_1

File: ros2_ws/src/robot_arm_moveit_config/config/robot_arm.ros2_control.xacro (robot description, xacro)
@@ -29,39 +29,4 @@
                 <state_interface name="velocity"/>
             </joint>
-            <joint name="joint_4">
-                <command_interface name="position"/>
-                <state_interface name="position">
-                  <param name="initial_value">${initial_positions['joint_4']}</param>
-                </state_interface>
-                <state_interface name="velocity"/>
-            </joint>
-            <joint name="joint_5">
-                <command_interface name="position"/>
-                <state_interface name="position">
-                  <param name="initial_value">${initial_positions['joint_5']}</param>
-                </state_interface>
-                <state_interface name="velocity"/>
-            </joint>
-            <joint name="joint_6">
-                <command_interface name="position"/>
-                <state_interface name="position">
-                  <param name="initial_value">${initial_positions['joint_6']}</param>
-                </state_interface>
-                <state_interface name="velocity"/>
-            </joint>
-            <joint name="left_finger_joint">
-                <command_interface name="position"/>
-                <state_interface name="position">
-                  <param name="initial_value">${initial_positions['left_finger_joint']}</param>
-                </state_interface>
-                <state_interface name="velocity"/>
-            </joint>
-            <joint name="right_finger_joint">
-                <command_interface name="position"/>
-                <state_interface name="position">
-                  <param name="initial_value">${initial_positions['right_finger_joint']}</param>
-                </state_interface>
-                <state_interface name="velocity"/>
-            </joint>
         </ros2_control>
     </xacro:macro>
