Commit message: fix(urdf): joint_3/joint_5 회전축을 주석 의도에 맞게 수정
joint_3은 팔꿈치 상하 굽힘(Y축)이어야 하나 Z축으로,
joint_5는 손목 비틀기(Z축, 링크 길이방향)여야 하나 Y축으로 설정돼
있어 RViz/MoveIt에서 팔이 의도와 다르게 움직였다.
- joint_3: axis 0 0 1 -> 0 1 0
- joint_5: axis 0 1 0 -> 0 0 1

Co-Authored-By: Claude Opus 4.7 <noreply@anthropic.com>

File: ros2_ws/src/robot_arm_description/urdf/robot_arm.urdf (robot description, URDF)
Before this commit: robot robot_arm, 10 links, 9 joints
Joints:
- joint joint_3: axis 0 0 1 -> 0 1 0
- joint joint_5: axis 0 1 0 -> 0 0 1

Commit message: feat(robot_arm_description): 2026-07-07 CAD export로 URDF/메시 교체 (5축)
- urdf/robot_arm.urdf를 새 CAD export(urdf_0707.urdf) 기반으로 교체, package 경로만
  robot_arm_description으로 수정. 링크/조인트 이름은 CAD 원본(한글, Revolute NN)을 유지.
  actuated joint 5개(Revolute 23/29/42/48/72), 그리퍼 없음 - 기존 6축+그리퍼 URDF와는
  다른 구조라 SRDF/controllers.yaml/moveit_dynamixel_bridge 쪽은 아직 안 맞음.
- meshes/ 전체를 새 CAD export의 STL 41개로 교체(기존 31개 삭제).
- Revolute 29 axis를 반전(+X -> -X)하고 limit을 [pi,2pi]에서 [-pi,0]으로 재라벨링해서
  실제 자세는 그대로 두고 joint_state_publisher의 기본값(0)이 기존 6.283 자리(정지 자세)에
  오도록 맞춤.
- display.launch.py의 joint_state_publisher를 joint_state_publisher_gui로 수정
  (문서에는 gui로 되어있었지만 실제 코드는 슬라이더 없는 버전이었음).

Co-Authored-By: Claude Sonnet 5 <noreply@anthropic.com>

File: ros2_ws/src/robot_arm_description/urdf/robot_arm.urdf (robot description, URDF)
Before this commit: robot robot_arm, 30 links, 29 joints
Links:
- removed link Adapter_A_1
- removed link Adapter_A_1_1
- removed link Adapter_B_1
- removed link Adapter_B_1_1_1
- removed link Adapter_b_1_1
- removed link Bottom_Cylinder_1
- removed link Bottom_top_1
- removed link GearBox1_1
- removed link GearBox2_1
- removed link Link1_1
- removed link Link1_1_1
- removed link Link2Bridge2_1
- removed link Link2Bridge_1
- removed link Link2_1
- removed link Link2_1_1
- removed link Link3Bridge2_1
- removed link Link3Bridge_1
- removed link Link3_1
- removed link Link3_1_1
- removed link Link4_1
- removed link Link4_1_1
- removed link Link5_1_1
- removed link Link_5_1
- removed link Motor0_1
- removed link Motor1_1
- removed link Motor2_1
- removed link Motor_1
- removed link Plug_1
- removed link _Plug2_1
- added link 5축_모듈_연결부_Component41_1, mass 1.9126732622839608; collision mesh filename=package://robot_arm_description/meshes/5축_모듈_연결부_Component4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 scale=0.001 0.001 0.001; visual mesh filename=package://robot_arm_description/meshes/5축_모듈_연결부_Component4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 scale=0.001 0.001 0.001
- added link Component38_1, mass 0.5585472030657777; collision mesh filename=package://robot_arm_description/meshes/Component38_1.stl scale=0.001 0.001 0.001; visual mesh filename=package://robot_arm_description/meshes/Component38_1.stl scale=0.001 0.001 0.001
- added link Component40_1, mass 0.6121227780764895; collision mesh filename=package://robot_arm_description/meshes/Component40_1.stl scale=0.001 0.001 0.001; visual mesh filename=package://robot_arm_description/meshes/Component40_1.stl scale=0.001 0.001 0.001
- added link XL430_T_1, mass 0.34622507558019666; collision mesh filename=package://robot_arm_description/meshes/XL430_T_1.stl scale=0.001 0.001 0.001; visual mesh filename=package://robot_arm_description/meshes/XL430_T_1.stl scale=0.001 0.001 0.001
- added link 기어박스1_1, mass 2.039024001006148; collision mesh filename=package://robot_arm_description/meshes/기어박스1_1.stl scale=0.001 0.001 0.001; visual mesh filename=package://robot_arm_description/meshes/기어박스1_1.stl scale=0.001 0.001 0.001
- added link 기어박스1__1__1, mass 2.0338757908094958; collision mesh filename=package://robot_arm_description/meshes/기어박스1__1__1.stl scale=0.001 0.001 0.001; visual mesh filename=package://robot_arm_description/meshes/기어박스1__1__1.stl scale=0.001 0.001 0.001
- added link 링크1-1_1, mass 0.40614905152898423; collision mesh filename=package://robot_arm_description/meshes/링크1-1_1.stl scale=0.001 0.001 0.001; visual mesh filename=package://robot_arm_description/meshes/링크1-1_1.stl scale=0.001 0.001 0.001
- added link 링크1_1, mass 0.44759500853450696; collision mesh filename=package://robot_arm_description/meshes/링크1_1.stl scale=0.001 0.001 0.001; visual mesh filename=package://robot_arm_description/meshes/링크1_1.stl scale=0.001 0.001 0.001
- added link 링크1__1__1, mass 0.1900850226097608; collision mesh filename=package://robot_arm_description/meshes/링크1__1__1.stl scale=0.001 0.001 0.001; visual mesh filename=package://robot_arm_description/meshes/링크1__1__1.stl scale=0.001 0.001 0.001
- added link 링크2-1__3__1, mass 0.5733792760793044; collision mesh filename=package://robot_arm_description/meshes/링크2-1__3__1.stl scale=0.001 0.001 0.001; visual mesh filename=package://robot_arm_description/meshes/링크2-1__3__1.stl scale=0.001 0.001 0.001
- added link 링크2_1, mass 0.5760752094127702; collision mesh filename=package://robot_arm_description/meshes/링크2_1.stl scale=0.001 0.001 0.001; visual mesh filename=package://robot_arm_description/meshes/링크2_1.stl scale=0.001 0.001 0.001
- added link 링크2__1__1, mass 0.20741862160121777; collision mesh filename=package://robot_arm_description/meshes/링크2__1__1.stl scale=0.001 0.001 0.001; visual mesh filename=package://robot_arm_description/meshes/링크2__1__1.stl scale=0.001 0.001 0.001
- added link 링크2다리2_1, mass 0.17597826669199707; collision mesh filename=package://robot_arm_description/meshes/링크2다리2_1.stl scale=0.001 0.001 0.001; visual mesh filename=package://robot_arm_description/meshes/링크2다리2_1.stl scale=0.001 0.001 0.001
- added link 링크2다리_1, mass 0.22700261556158713; collision mesh filename=package://robot_arm_description/meshes/링크2다리_1.stl scale=0.001 0.001 0.001; visual mesh filename=package://robot_arm_description/meshes/링크2다리_1.stl scale=0.001 0.001 0.001
- added link 링크3-1_1, mass 0.8186445791058825; collision mesh filename=package://robot_arm_description/meshes/링크3-1_1.stl scale=0.001 0.001 0.001; visual mesh filename=package://robot_arm_description/meshes/링크3-1_1.stl scale=0.001 0.001 0.001
- added link 링크3_1, mass 0.8034510771086975; collision mesh filename=package://robot_arm_description/meshes/링크3_1.stl scale=0.001 0.001 0.001; visual mesh filename=package://robot_arm_description/meshes/링크3_1.stl scale=0.001 0.001 0.001
- added link 링크3다리2_1, mass 0.2226363143753701; collision mesh filename=package://robot_arm_description/meshes/링크3다리2_1.stl scale=0.001 0.001 0.001; visual mesh filename=package://robot_arm_description/meshes/링크3다리2_1.stl scale=0.001 0.001 0.001
- added link 링크3다리_1, mass 0.3308579843753697; collision mesh filename=package://robot_arm_description/meshes/링크3다리_1.stl scale=0.001 0.001 0.001; visual mesh filename=package://robot_arm_description/meshes/링크3다리_1.stl scale=0.001 0.001 0.001
- added link 링크4-1_1, mass 0.21082599155250997; collision mesh filename=package://robot_arm_description/meshes/링크4-1_1.stl scale=0.001 0.001 0.001; visual mesh filename=package://robot_arm_description/meshes/링크4-1_1.stl scale=0.001 0.001 0.001
- added link 링크4_1, mass 0.21082599155250994; collision mesh filename=package://robot_arm_description/meshes/링크4_1.stl scale=0.001 0.001 0.001; visual mesh filename=package://robot_arm_description/meshes/링크4_1.stl scale=0.001 0.001 0.001
- added link 링크5-1_1, mass 0.24038547715832267; collision mesh filename=package://robot_arm_description/meshes/링크5-1_1.stl scale=0.001 0.001 0.001; visual mesh filename=package://robot_arm_description/meshes/링크5-1_1.stl scale=0.001 0.001 0.001
- added link 링크5_1, mass 0.2576677637629673; collision mesh filename=package://robot_arm_description/meshes/링크5_1.stl scale=0.001 0.001 0.001; visual mesh filename=package://robot_arm_description/meshes/링크5_1.stl scale=0.001 0.001 0.001
- added link 마개2_1, mass 0.12724315500067693; collision mesh filename=package://robot_arm_description/meshes/마개2_1.stl scale=0.001 0.001 0.001; visual mesh filename=package://robot_arm_description/meshes/마개2_1.stl scale=0.001 0.001 0.001
- added link 마개_1, mass 0.1272431550006768; collision mesh filename=package://robot_arm_description/meshes/마개_1.stl scale=0.001 0.001 0.001; visual mesh filename=package://robot_arm_description/meshes/마개_1.stl scale=0.001 0.001 0.001
- added link 모터0_1, mass 0.664027798614862; collision mesh filename=package://robot_arm_description/meshes/모터0_1.stl scale=0.001 0.001 0.001; visual mesh filename=package://robot_arm_description/meshes/모터0_1.stl scale=0.001 0.001 0.001
- added link 모터1_1, mass 0.6640277986148614; collision mesh filename=package://robot_arm_description/meshes/모터1_1.stl scale=0.001 0.001 0.001; visual mesh filename=package://robot_arm_description/meshes/모터1_1.stl scale=0.001 0.001 0.001
- added link 모터2_1, mass 0.6620566191194474; collision mesh filename=package://robot_arm_description/meshes/모터2_1.stl scale=0.001 0.001 0.001; visual mesh filename=package://robot_arm_description/meshes/모터2_1.stl scale=0.001 0.001 0.001
- added link 모터_1, mass 0.6640277986148609; collision mesh filename=package://robot_arm_description/meshes/모터_1.stl scale=0.001 0.001 0.001; visual mesh filename=package://robot_arm_description/meshes/모터_1.stl scale=0.001 0.001 0.001
- added link 바닥_1, mass 0.7527923586440036; collision mesh filename=package://robot_arm_description/meshes/바닥_1.stl scale=0.001 0.001 0.001; visual mesh filename=package://robot_arm_description/meshes/바닥_1.stl scale=0.001 0.001 0.001
- added link 상단_1, mass 0.11483450819161148; collision mesh filename=package://robot_arm_description/meshes/상단_1.stl scale=0.001 0.001 0.001; visual mesh filename=package://robot_arm_description/meshes/상단_1.stl scale=0.001 0.001 0.001
- added link 어댑터_1, mass 0.037276333994375375; collision mesh filename=package://robot_arm_description/meshes/어댑터_1.stl scale=0.001 0.001 0.001; visual mesh filename=package://robot_arm_description/meshes/어댑터_1.stl scale=0.001 0.001 0.001
- added link 어댑터a_1, mass 0.09838512042156757; collision mesh filename=package://robot_arm_description/meshes/어댑터a_1.stl scale=0.001 0.001 0.001; visual mesh filename=package://robot_arm_description/meshes/어댑터a_1.stl scale=0.001 0.001 0.001
- added link 어댑터a__1__1, mass 0.09838512042156751; collision mesh filename=package://robot_arm_description/meshes/어댑터a__1__1.stl scale=0.001 0.001 0.001; visual mesh filename=package://robot_arm_description/meshes/어댑터a__1__1.stl scale=0.001 0.001 0.001
- added link 어댑터b_1, mass 0.0383693503096125; collision mesh filename=package://robot_arm_description/meshes/어댑터b_1.stl scale=0.001 0.001 0.001; visual mesh filename=package://robot_arm_description/meshes/어댑터b_1.stl scale=0.001 0.001 0.001
- added link 어댑터b__1__1, mass 0.1507674746734739; collision mesh filename=package://robot_arm_description/meshes/어댑터b__1__1.stl scale=0.001 0.001 0.001; visual mesh filename=package://robot_arm_description/meshes/어댑터b__1__1.stl scale=0.001 0.001 0.001
- added link 어댑터b__1___1__1, mass 0.0836288961017048; collision mesh filename=package://robot_arm_description/meshes/어댑터b__1___1__1.stl scale=0.001 0.001 0.001; visual mesh filename=package://robot_arm_description/meshes/어댑터b__1___1__1.stl scale=0.001 0.001 0.001
- added link 연결부_1__1, mass 0.14836014599953082; collision mesh filename=package://robot_arm_description/meshes/연결부_1__1.stl scale=0.001 0.001 0.001; visual mesh filename=package://robot_arm_description/meshes/연결부_1__1.stl scale=0.001 0.001 0.001
- added link 파워트레인_1, mass 0.0024661502330680955; collision mesh filename=package://robot_arm_description/meshes/파워트레인_1.stl scale=0.001 0.001 0.001; visual mesh filename=package://robot_arm_description/meshes/파워트레인_1.stl scale=0.001 0.001 0.001
- added link 하단_1, mass 0.12615164501277876; collision mesh filename=package://robot_arm_description/meshes/하단_1.stl scale=0.001 0.001 0.001; visual mesh filename=package://robot_arm_description/meshes/하단_1.stl scale=0.001 0.001 0.001
- added link 하부원통_1, mass 2.7522236601038736; collision mesh filename=package://robot_arm_description/meshes/하부원통_1.stl scale=0.001 0.001 0.001; visual mesh filename=package://robot_arm_description/meshes/하부원통_1.stl scale=0.001 0.001 0.001
Joints:
- removed joint Rigid 23
- removed joint Rigid 42
- removed joint Rigid 48
- removed joint Rigid 5
- removed joint Rigid 54
- removed joint Rigid 55
- removed joint Rigid 56
- removed joint Rigid 57
- removed joint Rigid 58
- removed joint Rigid 59
- removed joint Rigid 60
- removed joint Rigid 61
- removed joint joint_1
- removed joint joint_2
- removed joint joint_3
- added joint Revolute 23: type continuous, parent 하부원통_1, child 바닥_1, origin xyz=0.0 0.0 0.0465 rpy=0 0 0, axis 0.0 0.0 1.0
- added joint Revolute 29: type revolute, parent 모터_1, child 어댑터b_1, origin xyz=0.0465 0.0 0.0 rpy=0 0 0, axis -1.0 0.0 0.0, limit lower=-3.141593 upper=0.0 effort=100 velocity=100
- added joint Revolute 42: type revolute, parent 기어박스1__1__1, child 마개2_1, origin xyz=-0.0755 0.0 0.0 rpy=0 0 0, axis -1.0 0.0 0.0, limit lower=0.0 upper=3.141593 effort=100 velocity=100
- added joint Revolute 48: type revolute, parent 링크5_1, child 어댑터_1, origin xyz=0.0001 -0.068917 0.0045 rpy=0 0 0, axis -1.0 0.0 0.0, limit lower=-1.570796 upper=1.570796 effort=100 velocity=100
- added joint Revolute 72: type continuous, parent XL430_T_1, child 연결부_1__1, origin xyz=0.0309 0.001644 -0.00525 rpy=0 0 0, axis -0.0 -1.0 0.0
- added joint Rigid 20: type fixed, parent base_link, child 모터0_1, origin xyz=0.0 0.0 0.004 rpy=0 0 0
- added joint Rigid 24: type fixed, parent 바닥_1, child 링크1-1_1, origin xyz=0.0 -0.01 0.0085 rpy=0 0 0
- added joint Rigid 25: type fixed, parent 바닥_1, child 링크1_1, origin xyz=0.0 -0.01 0.0085 rpy=0 0 0
- added joint Rigid 26: type fixed, parent 링크1-1_1, child 기어박스1_1, origin xyz=-0.06215 0.004643 0.06 rpy=0 0 0
- added joint Rigid 27: type fixed, parent 기어박스1_1, child 어댑터a_1, origin xyz=0.0675 -0.005731 0.0 rpy=0 0 0
- added joint Rigid 28: type fixed, parent 어댑터a_1, child 모터_1, origin xyz=0.0103 0.005544 -0.0045 rpy=0 0 0
- added joint Rigid 30: type fixed, parent 어댑터b_1, child Component40_1, origin xyz=0.0148 0.0 0.0 rpy=0 0 0
- added joint Rigid 31: type fixed, parent Component40_1, child 링크2_1, origin xyz=0.002 0.15 -0.001 rpy=0 0 0
- added joint Rigid 32: type fixed, parent 링크2_1, child 어댑터b__1__1, origin xyz=-0.002 0.143 0.061 rpy=0 0 0
- added joint Rigid 33: type fixed, parent 링크2_1, child 링크2다리2_1, origin xyz=0.002 0.013819 -0.047 rpy=0 0 0
- added joint Rigid 34: type fixed, parent Component40_1, child 링크2다리_1, origin xyz=0.002 0.135652 0.049 rpy=0 0 0
- added joint Rigid 35: type fixed, parent 링크2다리_1, child Component38_1, origin xyz=-0.1586 0.025 0.0 rpy=0 0 0
- added joint Rigid 36: type fixed, parent 링크2다리_1, child 링크2-1__3__1, origin xyz=-0.1586 0.0 0.0 rpy=0 0 0
- added joint Rigid 37: type fixed, parent 링크2-1__3__1, child 마개_1, origin xyz=-0.002 -0.135652 -0.049 rpy=0 0 0
- added joint Rigid 38: type fixed, parent 어댑터b__1__1, child 모터1_1, origin xyz=-0.0303 0.0 0.0 rpy=0 0 0
- added joint Rigid 39: type fixed, parent 모터1_1, child 어댑터a__1__1, origin xyz=-0.044 0.0 0.0 rpy=0 0 0
- added joint Rigid 40: type fixed, parent 어댑터a__1__1, child 기어박스1__1__1, origin xyz=-0.0407 0.0 0.0 rpy=0 0 0
- added joint Rigid 44: type fixed, parent 링크3_1, child 링크3다리_1, origin xyz=0.0 -0.10674 0.108 rpy=0 0 0
- added joint Rigid 66: type fixed, parent 상단_1, child 링크1__1__1, origin xyz=0.0819 0.0 0.0 rpy=0 0 0
- added joint Rigid 71: type fixed, parent 링크2__1__1, child XL430_T_1, origin xyz=0.01505 -0.100544 -0.00025 rpy=0 0 0
- added joint Rigid 73: type fixed, parent 연결부_1__1, child 5축_모듈_연결부_Component41_1, origin xyz=0.0 -0.0051 0.0 rpy=0 0 0
- joint Rigid 21: child Bottom_Cylinder_1 -> 하부원통_1; origin xyz=0.0 0.01 -0.0005 rpy=0 0 0 -> xyz=0.0 0.0 0.004 rpy=0 0 0
- joint Rigid 22: child Link1_1 -> 파워트레인_1; origin xyz=0.0 0.0 0.004 rpy=0 0 0 -> xyz=0.0 0.0 0.0465 rpy=0 0 0; parent Bottom_top_1 -> 하부원통_1
- joint Rigid 43: child Motor_1 -> 링크3_1; origin xyz=-0.0025 -0.004186 0.0 rpy=0 0 0 -> xyz=0.0165 0.0 0.0 rpy=0 0 0; parent Adapter_B_1 -> 마개2_1
- joint Rigid 45: child GearBox1_1 -> 링크3다리2_1; origin xyz=-0.0093 0.004186 0.0 rpy=0 0 0 -> xyz=0.0 -0.10674 0.012 rpy=0 0 0; parent Adapter_A_1 -> 링크3_1
- joint Rigid 46: child Plug_1 -> 링크4_1; origin xyz=-0.1045 -0.004186 0.0 rpy=0 0 0 -> xyz=0.0 -0.194627 0.06 rpy=0 0 0; parent GearBox1_1 -> 링크3_1
- joint Rigid 47: child Link2_1_1 -> 링크5_1; origin xyz=0.0165 0.0 0.0 rpy=0 0 0 -> xyz=0.06865 0.0 0.0 rpy=0 0 0; parent Plug_1 -> 링크4_1
- joint Rigid 49: child Link2_1 -> 모터2_1; origin xyz=0.1626 0.0 0.0 rpy=0 0 0 -> xyz=0.0039 0.005544 -0.0045 rpy=0 0 0; parent Link2Bridge_1 -> 어댑터_1
- joint Rigid 50: child Link2Bridge2_1 -> 링크2__1__1; origin xyz=0.0 0.0175 -0.092 rpy=0 0 0 -> xyz=-0.0067 0.005544 0.006 rpy=0 0 0; parent Link2_1 -> 어댑터_1
- joint Rigid 51: child Adapter_b_1_1 -> 상단_1; origin xyz=-0.004 0.144849 0.014 rpy=0 0 0 -> xyz=-0.005 -0.094 0.0035 rpy=0 0 0; parent Link2_1 -> 링크2__1__1
- joint Rigid 52: child Motor1_1 -> 하단_1; origin xyz=-0.0288 0.0 0.0 rpy=0 0 0 -> xyz=-0.005 -0.094 -0.013 rpy=0 0 0; parent Adapter_b_1_1 -> 링크2__1__1
- joint Rigid 62: child Motor2_1 -> 링크3-1_1; origin xyz=0.004 -0.063373 0.0 rpy=0 0 0 -> xyz=0.1943 0.0 0.0 rpy=0 0 0; parent Link_5_1 -> 링크3다리_1
- joint Rigid 63: child Adapter_B_1_1_1 -> 링크4-1_1; origin xyz=0.0455 0.0 0.0 rpy=0 0 0 -> xyz=0.0 -0.087887 -0.048 rpy=0 0 0; parent Motor2_1 -> 링크3-1_1
- joint Rigid 64: child Link5_1_1 -> 링크5-1_1; origin xyz=0.0074 0.004186 0.0 rpy=0 0 0 -> xyz=-0.06865 0.0 0.0 rpy=0 0 0; parent Adapter_B_1_1_1 -> 링크4-1_1
- joint Rigid 65: child Link4_1_1 -> 어댑터b__1___1__1; origin xyz=0.0 0.059187 0.0 rpy=0 0 0 -> xyz=0.0001 -0.068917 0.0045 rpy=0 0 0; parent Link5_1_1 -> 링크5-1_1
