Commit message: fix(robot_arm_description): URDF/메시 링크 이름 한글 → 영어 변경
CAD export 원본 한글 링크 이름(모터_1, 링크2다리_1, 어댑터b__1__1 등)이
인코딩 문제로 깨지는 걸 방지하기 위해 동일한 의미의 영어 이름으로 변경.
CAD 인스턴스 접미사(__1__ 등)는 그대로 보존. joint 이름(Revolute NN 등)과
SRDF/controllers.yaml 등 다른 파일은 기존에 이미 안 맞는 상태(§8)라 손대지 않음.

meshes/ STL 35개는 git mv로 리네임해 히스토리 보존.
colcon build + xacro/check_urdf 파싱 + MoveIt mock demo(demo.launch.py) 실행으로 검증 완료.

Co-Authored-By: Claude Sonnet 5 <noreply@anthropic.com>

File: ros2_ws/src/robot_arm_description/urdf/robot_arm.urdf (robot description, URDF)
Before this commit: robot robot_arm, 41 links, 40 joints
Links:
- removed link 5축_모듈_연결부_Component41_1
- removed link 기어박스1_1
- removed link 기어박스1__1__1
- removed link 링크1-1_1
- removed link 링크1_1
- removed link 링크1__1__1
- removed link 링크2-1__3__1
- removed link 링크2_1
- removed link 링크2__1__1
- removed link 링크2다리2_1
- removed link 링크2다리_1
- removed link 링크3-1_1
- removed link 링크3_1
- removed link 링크3다리2_1
- removed link 링크3다리_1
- removed link 링크4-1_1
- removed link 링크4_1
- removed link 링크5-1_1
- removed link 링크5_1
- removed link 마개2_1
- removed link 마개_1
- removed link 모터0_1
- removed link 모터1_1
- removed link 모터2_1
- removed link 모터_1
- removed link 바닥_1
- removed link 상단_1
- removed link 어댑터_1
- removed link 어댑터a_1
- removed link 어댑터a__1__1
- removed link 어댑터b_1
- removed link 어댑터b__1__1
- removed link 어댑터b__1___1__1
- removed link 연결부_1__1
- removed link 파워트레인_1
- removed link 하단_1
- removed link 하부원통_1
- added link adapter_1, mass 0.037276333994375375; collision mesh filename=package://robot_arm_description/meshes/adapter_1.stl scale=0.001 0.001 0.001; visual mesh filename=package://robot_arm_description/meshes/adapter_1.stl scale=0.001 0.001 0.001
- added link adapter_a_1, mass 0.09838512042156757; collision mesh filename=package://robot_arm_description/meshes/adapter_a_1.stl scale=0.001 0.001 0.001; visual mesh filename=package://robot_arm_description/meshes/adapter_a_1.stl scale=0.001 0.001 0.001
- added link adapter_a__1__1, mass 0.09838512042156751; collision mesh filename=package://robot_arm_description/meshes/adapter_a__1__1.stl scale=0.001 0.001 0.001; visual mesh filename=package://robot_arm_description/meshes/adapter_a__1__1.stl scale=0.001 0.001 0.001
- added link adapter_b_1, mass 0.0383693503096125; collision mesh filename=package://robot_arm_description/meshes/adapter_b_1.stl scale=0.001 0.001 0.001; visual mesh filename=package://robot_arm_description/meshes/adapter_b_1.stl scale=0.001 0.001 0.001
- added link adapter_b__1__1, mass 0.1507674746734739; collision mesh filename=package://robot_arm_description/meshes/adapter_b__1__1.stl scale=0.001 0.001 0.001; visual mesh filename=package://robot_arm_description/meshes/adapter_b__1__1.stl scale=0.001 0.001 0.001
- added link adapter_b__1___1__1, mass 0.0836288961017048; collision mesh filename=package://robot_arm_description/meshes/adapter_b__1___1__1.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 scale=0.001 0.001 0.001; visual mesh filename=package://robot_arm_description/meshes/adapter_b__1___1__1.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 scale=0.001 0.001 0.001
- added link base_plate_1, mass 0.7527923586440036; collision mesh filename=package://robot_arm_description/meshes/base_plate_1.stl scale=0.001 0.001 0.001; visual mesh filename=package://robot_arm_description/meshes/base_plate_1.stl scale=0.001 0.001 0.001
- added link bottom_1, mass 0.12615164501277876; collision mesh filename=package://robot_arm_description/meshes/bottom_1.stl scale=0.001 0.001 0.001; visual mesh filename=package://robot_arm_description/meshes/bottom_1.stl scale=0.001 0.001 0.001
- added link cap2_1, mass 0.12724315500067693; collision mesh filename=package://robot_arm_description/meshes/cap2_1.stl scale=0.001 0.001 0.001; visual mesh filename=package://robot_arm_description/meshes/cap2_1.stl scale=0.001 0.001 0.001
- added link cap_1, mass 0.1272431550006768; collision mesh filename=package://robot_arm_description/meshes/cap_1.stl scale=0.001 0.001 0.001; visual mesh filename=package://robot_arm_description/meshes/cap_1.stl scale=0.001 0.001 0.001
- added link connector_1__1, mass 0.14836014599953082; collision mesh filename=package://robot_arm_description/meshes/connector_1__1.stl scale=0.001 0.001 0.001; visual mesh filename=package://robot_arm_description/meshes/connector_1__1.stl scale=0.001 0.001 0.001
- added link gearbox1_1, mass 2.039024001006148; collision mesh filename=package://robot_arm_description/meshes/gearbox1_1.stl scale=0.001 0.001 0.001; visual mesh filename=package://robot_arm_description/meshes/gearbox1_1.stl scale=0.001 0.001 0.001
- added link gearbox1__1__1, mass 2.0338757908094958; collision mesh filename=package://robot_arm_description/meshes/gearbox1__1__1.stl scale=0.001 0.001 0.001; visual mesh filename=package://robot_arm_description/meshes/gearbox1__1__1.stl scale=0.001 0.001 0.001
- added link link1-1_1, mass 0.40614905152898423; collision mesh filename=package://robot_arm_description/meshes/link1-1_1.stl scale=0.001 0.001 0.001; visual mesh filename=package://robot_arm_description/meshes/link1-1_1.stl scale=0.001 0.001 0.001
- added link link1_1, mass 0.44759500853450696; collision mesh filename=package://robot_arm_description/meshes/link1_1.stl scale=0.001 0.001 0.001; visual mesh filename=package://robot_arm_description/meshes/link1_1.stl scale=0.001 0.001 0.001
- added link link1__1__1, mass 0.1900850226097608; collision mesh filename=package://robot_arm_description/meshes/link1__1__1.stl scale=0.001 0.001 0.001; visual mesh filename=package://robot_arm_description/meshes/link1__1__1.stl scale=0.001 0.001 0.001
- added link link2-1__3__1, mass 0.5733792760793044; collision mesh filename=package://robot_arm_description/meshes/link2-1__3__1.stl scale=0.001 0.001 0.001; visual mesh filename=package://robot_arm_description/meshes/link2-1__3__1.stl scale=0.001 0.001 0.001
- added link link2_1, mass 0.5760752094127702; collision mesh filename=package://robot_arm_description/meshes/link2_1.stl scale=0.001 0.001 0.001; visual mesh filename=package://robot_arm_description/meshes/link2_1.stl scale=0.001 0.001 0.001
- added link link2__1__1, mass 0.20741862160121777; collision mesh filename=package://robot_arm_description/meshes/link2__1__1.stl scale=0.001 0.001 0.001; visual mesh filename=package://robot_arm_description/meshes/link2__1__1.stl scale=0.001 0.001 0.001
- added link link2_leg2_1, mass 0.17597826669199707; collision mesh filename=package://robot_arm_description/meshes/link2_leg2_1.stl scale=0.001 0.001 0.001; visual mesh filename=package://robot_arm_description/meshes/link2_leg2_1.stl scale=0.001 0.001 0.001
- added link link2_leg_1, mass 0.22700261556158713; collision mesh filename=package://robot_arm_description/meshes/link2_leg_1.stl scale=0.001 0.001 0.001; visual mesh filename=package://robot_arm_description/meshes/link2_leg_1.stl scale=0.001 0.001 0.001
- added link link3-1_1, mass 0.8186445791058825; collision mesh filename=package://robot_arm_description/meshes/link3-1_1.stl scale=0.001 0.001 0.001; visual mesh filename=package://robot_arm_description/meshes/link3-1_1.stl scale=0.001 0.001 0.001
- added link link3_1, mass 0.8034510771086975; collision mesh filename=package://robot_arm_description/meshes/link3_1.stl scale=0.001 0.001 0.001; visual mesh filename=package://robot_arm_description/meshes/link3_1.stl scale=0.001 0.001 0.001
- added link link3_leg2_1, mass 0.2226363143753701; collision mesh filename=package://robot_arm_description/meshes/link3_leg2_1.stl scale=0.001 0.001 0.001; visual mesh filename=package://robot_arm_description/meshes/link3_leg2_1.stl scale=0.001 0.001 0.001
- added link link3_leg_1, mass 0.3308579843753697; collision mesh filename=package://robot_arm_description/meshes/link3_leg_1.stl scale=0.001 0.001 0.001; visual mesh filename=package://robot_arm_description/meshes/link3_leg_1.stl scale=0.001 0.001 0.001
- added link link4-1_1, mass 0.21082599155250997; collision mesh filename=package://robot_arm_description/meshes/link4-1_1.stl scale=0.001 0.001 0.001; visual mesh filename=package://robot_arm_description/meshes/link4-1_1.stl scale=0.001 0.001 0.001
- added link link4_1, mass 0.21082599155250994; collision mesh filename=package://robot_arm_description/meshes/link4_1.stl scale=0.001 0.001 0.001; visual mesh filename=package://robot_arm_description/meshes/link4_1.stl scale=0.001 0.001 0.001
- added link link5-1_1, mass 0.24038547715832267; collision mesh filename=package://robot_arm_description/meshes/link5-1_1.stl scale=0.001 0.001 0.001; visual mesh filename=package://robot_arm_description/meshes/link5-1_1.stl scale=0.001 0.001 0.001
- added link link5_1, mass 0.2576677637629673; collision mesh filename=package://robot_arm_description/meshes/link5_1.stl scale=0.001 0.001 0.001; visual mesh filename=package://robot_arm_description/meshes/link5_1.stl scale=0.001 0.001 0.001
- added link lower_cylinder_1, mass 2.7522236601038736; collision mesh filename=package://robot_arm_description/meshes/lower_cylinder_1.stl scale=0.001 0.001 0.001; visual mesh filename=package://robot_arm_description/meshes/lower_cylinder_1.stl scale=0.001 0.001 0.001
- added link module_connector_5axis_Component41_1, mass 1.9126732622839608; collision mesh filename=package://robot_arm_description/meshes/module_connector_5ax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 scale=0.001 0.001 0.001; visual mesh filename=package://robot_arm_description/meshes/module_connector_5ax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 scale=0.001 0.001 0.001
- added link motor0_1, mass 0.664027798614862; collision mesh filename=package://robot_arm_description/meshes/motor0_1.stl scale=0.001 0.001 0.001; visual mesh filename=package://robot_arm_description/meshes/motor0_1.stl scale=0.001 0.001 0.001
- added link motor1_1, mass 0.6640277986148614; collision mesh filename=package://robot_arm_description/meshes/motor1_1.stl scale=0.001 0.001 0.001; visual mesh filename=package://robot_arm_description/meshes/motor1_1.stl scale=0.001 0.001 0.001
- added link motor2_1, mass 0.6620566191194474; collision mesh filename=package://robot_arm_description/meshes/motor2_1.stl scale=0.001 0.001 0.001; visual mesh filename=package://robot_arm_description/meshes/motor2_1.stl scale=0.001 0.001 0.001
- added link motor_1, mass 0.6640277986148609; collision mesh filename=package://robot_arm_description/meshes/motor_1.stl scale=0.001 0.001 0.001; visual mesh filename=package://robot_arm_description/meshes/motor_1.stl scale=0.001 0.001 0.001
- added link powertrain_1, mass 0.0024661502330680955; collision mesh filename=package://robot_arm_description/meshes/powertrain_1.stl scale=0.001 0.001 0.001; visual mesh filename=package://robot_arm_description/meshes/powertrain_1.stl scale=0.001 0.001 0.001
- added link top_1, mass 0.11483450819161148; collision mesh filename=package://robot_arm_description/meshes/top_1.stl scale=0.001 0.001 0.001; visual mesh filename=package://robot_arm_description/meshes/top_1.stl scale=0.001 0.001 0.001
Joints:
- joint Revolute 23: child 바닥_1 -> base_plate_1; parent 하부원통_1 -> lower_cylinder_1
- joint Revolute 29: child 어댑터b_1 -> adapter_b_1; parent 모터_1 -> motor_1
- joint Revolute 42: child 마개2_1 -> cap2_1; parent 기어박스1__1__1 -> gearbox1__1__1
- joint Revolute 48: child 어댑터_1 -> adapter_1; parent 링크5_1 -> link5_1
- joint Revolute 72: child 연결부_1__1 -> connector_1__1
- joint Rigid 20: child 모터0_1 -> motor0_1
- joint Rigid 21: child 하부원통_1 -> lower_cylinder_1
- joint Rigid 22: child 파워트레인_1 -> powertrain_1; parent 하부원통_1 -> lower_cylinder_1
- joint Rigid 24: child 링크1-1_1 -> link1-1_1; parent 바닥_1 -> base_plate_1
- joint Rigid 25: child 링크1_1 -> link1_1; parent 바닥_1 -> base_plate_1
- joint Rigid 26: child 기어박스1_1 -> gearbox1_1; parent 링크1-1_1 -> link1-1_1
- joint Rigid 27: child 어댑터a_1 -> adapter_a_1; parent 기어박스1_1 -> gearbox1_1
- joint Rigid 28: child 모터_1 -> motor_1; parent 어댑터a_1 -> adapter_a_1
- joint Rigid 30: parent 어댑터b_1 -> adapter_b_1
- joint Rigid 31: child 링크2_1 -> link2_1
- joint Rigid 32: child 어댑터b__1__1 -> adapter_b__1__1; parent 링크2_1 -> link2_1
- joint Rigid 33: child 링크2다리2_1 -> link2_leg2_1; parent 링크2_1 -> link2_1
- joint Rigid 34: child 링크2다리_1 -> link2_leg_1
- joint Rigid 35: parent 링크2다리_1 -> link2_leg_1
- joint Rigid 36: child 링크2-1__3__1 -> link2-1__3__1; parent 링크2다리_1 -> link2_leg_1
- joint Rigid 37: child 마개_1 -> cap_1; parent 링크2-1__3__1 -> link2-1__3__1
- joint Rigid 38: child 모터1_1 -> motor1_1; parent 어댑터b__1__1 -> adapter_b__1__1
- joint Rigid 39: child 어댑터a__1__1 -> adapter_a__1__1; parent 모터1_1 -> motor1_1
- joint Rigid 40: child 기어박스1__1__1 -> gearbox1__1__1; parent 어댑터a__1__1 -> adapter_a__1__1
- joint Rigid 43: child 링크3_1 -> link3_1; parent 마개2_1 -> cap2_1
- joint Rigid 44: child 링크3다리_1 -> link3_leg_1; parent 링크3_1 -> link3_1
- joint Rigid 45: child 링크3다리2_1 -> link3_leg2_1; parent 링크3_1 -> link3_1
- joint Rigid 46: child 링크4_1 -> link4_1; parent 링크3_1 -> link3_1
- joint Rigid 47: child 링크5_1 -> link5_1; parent 링크4_1 -> link4_1
- joint Rigid 49: child 모터2_1 -> motor2_1; parent 어댑터_1 -> adapter_1
- joint Rigid 50: child 링크2__1__1 -> link2__1__1; parent 어댑터_1 -> adapter_1
- joint Rigid 51: child 상단_1 -> top_1; parent 링크2__1__1 -> link2__1__1
- joint Rigid 52: child 하단_1 -> bottom_1; parent 링크2__1__1 -> link2__1__1
- joint Rigid 62: child 링크3-1_1 -> link3-1_1; parent 링크3다리_1 -> link3_leg_1
- joint Rigid 63: child 링크4-1_1 -> link4-1_1; parent 링크3-1_1 -> link3-1_1
- joint Rigid 64: child 링크5-1_1 -> link5-1_1; parent 링크4-1_1 -> link4-1_1
- joint Rigid 65: child 어댑터b__1___1__1 -> adapter_b__1___1__1; parent 링크5-1_1 -> link5-1_1
- joint Rigid 66: child 링크1__1__1 -> link1__1__1; parent 상단_1 -> top_1
- joint Rigid 71: parent 링크2__1__1 -> link2__1__1
- joint Rigid 73: child 5축_모듈_연결부_Component41_1 -> module_connector_5axis_Component41_1; parent 연결부_1__1 -> connector_1__1

Commit message: feat(teleop): 조이스틱 벤치 텔레옵 — 파워트레인 없이 팔 5축 구동
파워트레인 계약을 다 맞추려면 접힘 자세 → STOWED_LOCKED → SRDF 5축 재생성 →
MoveIt Servo 순으로 긴 체인을 타야 한다. 그 전에 팔을 실제로 움직여 본다.

## 격리 — 코드 분기 0줄

텔레옵 경로가 쓰는 토픽은 /arm/teleop_*, /joint_states, /dynamixel/goal_position
뿐이고 계약 토픽(/arm_status, /chassis_mode, /arrival_status)을 하나도 안 건드린다.
그것들은 arm_fsm 만 쓴다.

→ bench.launch.py 가 arm_fsm 을 안 띄우는 것으로 격리가 끝난다. 노드 코드에
"테스트 모드면 건너뛰기" 분기는 넣지 않았다 — 안전 게이트에 스킵 분기가 있으면
실기에서 켜진 채 도는 사고가 언젠가 난다.
검증: bench.launch.py 기동 시 계약 토픽이 아예 생기지 않음을 확인.

## main 의 URDF 가 깨져 있었다

main 의 robot_arm.urdf 는 관절 이름이 raw CAD 이름(Revolute 23~72)이고 그중 둘은
continuous(제한 없음)였다. 반면 position_node·arm_fsm 은 joint_1~joint_5 를 쓴다
→ 이름이 안 맞아 RViz 가 안 움직이고 joint_1/joint_5 는 무한 회전한다.
feat/teleop-keyboard 의 수정본(joint_1~5 + revolute 제한)을 가져왔다.

## teleop_core — velocities 를 rad/s 로

기존: goal += v * jog_step_rad * dt → 풀스틱(v=1.0)이 0.05 rad/s. joint_1 한 바퀴에
126초로 사실상 안 움직였다. JointJog.velocities 는 관례상 rad/s 다.

- goal += v * dt 로 수정
- max_vel_rad_s(기본 1.0) 신설 — 프론트엔드 버그로 큰 값이 와도 팔이 튀지 않게
- 키보드는 displacements 만 쓰므로 영향 없음 (회귀 확인: 3 x 0.05 = 0.15 정확)

## joystick_teleop_node — 5축 직접 매핑

L1=데드맨, 왼스틱=joint_1/2, 오른스틱=joint_3/4, L3/R3=joint_5,
R1=터보, △=home, ○=stop, ✕=비상정지(latched), PS=DRIVE/ARM 전환(스텁).

안전 장치:
- /joy 콜백이 아니라 자체 타이머(20Hz)에서 발행 — 스틱을 붙들고 있어도 메시지가
  끊기지 않게(끊기면 teleop_core 데드맨이 팔을 세운다)
- /joy 신선도 감시(0.5s) — 패드를 뽑아도 마지막 축 값을 재발행하지 않아 폭주 없음
- 매 발행마다 전 관절을 싣고 velocity 를 0 포함해 채움 — 일부만 보내면 놓은 관절이
  마지막 속도로 계속 돈다(teleop_core.on_jog 가 없는 관절을 0으로 만들지 않음)
- 데드존(0.15), 버튼 edge-trigger

## 그리퍼는 제외 (판단)

하드웨어는 동작한다(HW-8 검증). 빼는 이유는 소유권 중복이다 —
moveit_dynamixel_bridge 가 이미 같은 서보(id 5)를 구동하므로 position_node 에도
넣으면 같은 버스의 같은 서보를 두 노드가 서로 다른 표현으로 만지게 된다.
게다가 표현이 세 갈래(URDF continuous / 브릿지 prismatic 미터 / HW 스크립트 degree)로
갈라져 있다. 먼저 한 곳으로 정리한 뒤 배선할 것. 키맵 자리만 예약했다.

⚠️ 배선할 사람을 위해: Profile Acceleration(108)/Velocity(112) 를 25/80 으로 설정할 것.
기본값 0(=최고속 즉시 이동)이면 움직일 때마다 과전류로 토크가 풀린다
(HW-8, 재현율 100%, 0.3초 내 트립). CLAUDE.md 에 기록.

## 검증 (가짜 /joy 로 패드 없이 end-to-end)

- 데드맨(L1) 미보유 + 스틱 최대 → /dynamixel/goal_position 발행 0건
- 데드맨 보유 → 5축이 각각 자기 관절만 이동 (joint_1~5 전부 확인)
- velocity 가 실제 rad/s: 0.6 rad/s x 2.15s = 1.29 rad 이동 확인
  (수정 전 코드였다면 0.006 rad)
- 소프트 리밋: joint_4 가 정확히 π/2(1.5707963)에서, joint_2 가 상한 0.0 에서 정지
- 패드 사망: /joy 를 끊어도 3초간 미동 없음 (폭주 없음)
- 격리: 계약 토픽 0개
- 키보드 회귀 없음
- 패드 없이도 joy_node 포함 launch 정상 기동

Co-Authored-By: Claude Opus 4.8 (1M context) <noreply@anthropic.com>

File: ros2_ws/src/robot_arm_description/urdf/robot_arm.urdf (robot description, URDF)
Before this commit: robot robot_arm, 41 links, 40 joints
Joints:
- removed joint Revolute 23
- removed joint Revolute 29
- removed joint Revolute 42
- removed joint Revolute 48
- removed joint Revolute 72
- added joint joint_1: type revolute, parent lower_cylinder_1, child base_plate_1, origin xyz=0.0 0.0 0.0465 rpy=0 0 0, axis 0.0 0.0 1.0, limit lower=-3.141593 upper=3.141593 effort=100 velocity=100
- added joint joint_2: type revolute, parent motor_1, child adapter_b_1, origin xyz=0.0465 0.0 0.0 rpy=0 0 0, axis -1.0 0.0 0.0, limit lower=-3.141593 upper=0.0 effort=100 velocity=100
- added joint joint_3: type revolute, parent gearbox1__1__1, child cap2_1, origin xyz=-0.0755 0.0 0.0 rpy=0 0 0, axis -1.0 0.0 0.0, limit lower=0.0 upper=3.141593 effort=100 velocity=100
- added joint joint_4: type revolute, parent link5_1, child adapter_1, origin xyz=0.0001 -0.068917 0.0045 rpy=0 0 0, axis -1.0 0.0 0.0, limit lower=-1.570796 upper=1.570796 effort=100 velocity=100
- added joint joint_5: type revolute, parent XL430_T_1, child connector_1__1, origin xyz=0.0309 0.001644 -0.00525 rpy=0 0 0, axis -0.0 -1.0 0.0, limit lower=-3.141593 upper=3.141593 effort=100 velocity=100
