Commit message: feat(robot_arm_description): Isaac Sim export로 팔+그리퍼 URDF 전면 교체
RViz에서 팔 2/3축이 계속 이상하게 보이는 문제가 있었음. 원인을 진단해보니 기존
Fusion360 fusion2urdf 계열(VerNOmiddle) export의 joint_2 축 부호가 실제와
반대였고, 그 아래 매달린 3축 이하가 덩달아 이상해 보인 것이었음. 사용자가 이
CAD 파이프라인 자체를 신뢰하기 어렵다고 판단해, Isaac Sim에서 새로 뽑은
robotarm_urdf_20260711.urdf(+closed_loop.usd)로 URDF를 통째로 교체하기로 결정.

- mesh 58개: 원본에 딸린 meshes_ascii STL이 실제로는 어디에도 없어서(Isaac Sim
  exporter가 geometry를 USD에만 남김), usd-core(pxr)로 USD 안의 raw mesh point를
  직접 추출 → numpy-stl로 binary STL 변환 → robot_arm_description/meshes/ 전체
  교체(기존 56개 mesh, gripper_a 서브트리 포함 전량 대체).
- 그리퍼가 이제 실제 구동 조인트 gripper_drive_joint 하나 + URDF <mimic> 태그로
  종속되는 8개(크랭크/조 관절)로 정식 표현됨 — 기존엔 평행 4절링크의 닫힌 루프를
  중복 링크를 잘라내는 방식으로 근사해 실제 기구 구속을 못 담았음.
- 조인트 이름 체계 변경(joint_1~5, gripper_a_joint5/6 → arm_joint_1~5,
  gripper_drive_joint)을 dynamixel_control(moveit_dynamixel_bridge.py의
  JOINT_CONFIG, arm_fsm_node.py의 ARM_JOINT_NAMES/tip_link 기본값,
  gripper_presets.py의 gripper_joints)과 robot_arm_moveit_config 전체(SRDF
  chain/group/group_state/end_effector/disable_collisions, joint_limits.yaml,
  initial_positions.yaml, moveit_controllers.yaml, ros2_controllers.yaml,
  robot_arm.ros2_control.xacro)에 걸쳐 갱신.
- SRDF disable_collisions는 새 58-link 토폴로지의 Adjacent(부모-자식) 쌍만
  URDF에서 프로그램적으로 자동 도출해 채움 — 기어 치합 등 자세무관 Default 쌍은
  실제 충돌체크 없이 지어내지 않고 비워둠(MoveIt Setup Assistant 재실행 필요,
  주석으로 명시).
- 레거시 dynamixel_position_node.py(별도 P-control 파이프라인, joint_1~3 이름
  그대로)는 범위 밖으로 판단해 의도적으로 안 건드림.

컨테이너에서 colcon build + display.launch.py로 전체 링크 로드, mimic 조인트
자동 종속 확인, 사용자가 RViz 육안으로도 확인 완료.

Co-Authored-By: Claude Sonnet 5 <noreply@anthropic.com>

File: ros2_ws/src/robot_arm_description/urdf/robot_arm.urdf (robot description, URDF)
Before this commit: robot robot_arm, 41 links, 40 joints
Links:
- removed link Component38_1
- removed link Component40_1
- removed link XL430_T_1
- removed link adapter_1
- removed link adapter_a_1
- removed link adapter_a__1__1
- removed link adapter_b_1
- removed link adapter_b__1__1
- removed link adapter_b__1___1__1
- removed link base_plate_1
- removed link bottom_1
- removed link cap2_1
- removed link cap_1
- removed link connector_1__1
- removed link gearbox1_1
- removed link gearbox1__1__1
- removed link link1-1_1
- removed link link1_1
- removed link link1__1__1
- removed link link2-1__3__1
- removed link link2_1
- removed link link2__1__1
- removed link link2_leg2_1
- removed link link2_leg_1
- removed link link3-1_1
- removed link link3_1
- removed link link3_leg2_1
- removed link link3_leg_1
- removed link link4-1_1
- removed link link4_1
- removed link link5-1_1
- removed link link5_1
- removed link lower_cylinder_1
- removed link module_connector_5axis_Component41_1
- removed link motor0_1
- removed link motor1_1
- removed link motor2_1
- removed link motor_1
- removed link powertrain_1
- removed link top_1
- added link link_001, mass 0.15394987554690048; collision mesh filename=package://robot_arm_description/meshes/link_001.stl scale=0.001 0.001 0.001; visual mesh filename=package://robot_arm_description/meshes/link_001.stl scale=0.001 0.001 0.001
- added link link_002, mass 0.19814051788719486; collision mesh filename=package://robot_arm_description/meshes/link_002.stl scale=0.001 0.001 0.001; visual mesh filename=package://robot_arm_description/meshes/link_002.stl scale=0.001 0.001 0.001
- added link link_003, mass 0.13969457823289902; collision mesh filename=package://robot_arm_description/meshes/link_003.stl scale=0.001 0.001 0.001; visual mesh filename=package://robot_arm_description/meshes/link_003.stl scale=0.001 0.001 0.001
- added link link_004, mass 0.27634623034311884; collision mesh filename=package://robot_arm_description/meshes/link_004.stl scale=0.001 0.001 0.001; visual mesh filename=package://robot_arm_description/meshes/link_004.stl scale=0.001 0.001 0.001
- added link link_005, mass 0.28157202083896593; collision mesh filename=package://robot_arm_description/meshes/link_005.stl scale=0.001 0.001 0.001; visual mesh filename=package://robot_arm_description/meshes/link_005.stl scale=0.001 0.001 0.001
- added link link_006, mass 0.08862458116688048; collision mesh filename=package://robot_arm_description/meshes/link_006.stl scale=0.001 0.001 0.001; visual mesh filename=package://robot_arm_description/meshes/link_006.stl scale=0.001 0.001 0.001
- added link link_007, mass 0.08268035520095174; collision mesh filename=package://robot_arm_description/meshes/link_007.stl scale=0.001 0.001 0.001; visual mesh filename=package://robot_arm_description/meshes/link_007.stl scale=0.001 0.001 0.001
- added link link_008, mass 0.07251339836837921; collision mesh filename=package://robot_arm_description/meshes/link_008.stl scale=0.001 0.001 0.001; visual mesh filename=package://robot_arm_description/meshes/link_008.stl scale=0.001 0.001 0.001
- added link link_009, mass 0.07251339836837922; collision mesh filename=package://robot_arm_description/meshes/link_009.stl scale=0.001 0.001 0.001; visual mesh filename=package://robot_arm_description/meshes/link_009.stl scale=0.001 0.001 0.001
- added link link_010, mass 0.19211177685064962; collision mesh filename=package://robot_arm_description/meshes/link_010.stl scale=0.001 0.001 0.001; visual mesh filename=package://robot_arm_description/meshes/link_010.stl scale=0.001 0.001 0.001
- added link link_011, mass 0.19721325419288177; collision mesh filename=package://robot_arm_description/meshes/link_011.stl scale=0.001 0.001 0.001; visual mesh filename=package://robot_arm_description/meshes/link_011.stl scale=0.001 0.001 0.001
- added link link_012, mass 0.21053904468872886; collision mesh filename=package://robot_arm_description/meshes/link_012.stl scale=0.001 0.001 0.001; visual mesh filename=package://robot_arm_description/meshes/link_012.stl scale=0.001 0.001 0.001
- added link link_013, mass 0.10912049174690072; collision mesh filename=package://robot_arm_description/meshes/link_013.stl scale=0.001 0.001 0.001; visual mesh filename=package://robot_arm_description/meshes/link_013.stl scale=0.001 0.001 0.001
- added link link_014, mass 0.016167745903671614; collision mesh filename=package://robot_arm_description/meshes/link_014.stl scale=0.001 0.001 0.001; visual mesh filename=package://robot_arm_description/meshes/link_014.stl scale=0.001 0.001 0.001
- added link link_015, mass 0.006305281770624219; collision mesh filename=package://robot_arm_description/meshes/link_015.stl scale=0.001 0.001 0.001; visual mesh filename=package://robot_arm_description/meshes/link_015.stl scale=0.001 0.001 0.001
- added link link_016, mass 1.2987414019147439; collision mesh filename=package://robot_arm_description/meshes/link_016.stl scale=0.001 0.001 0.001; visual mesh filename=package://robot_arm_description/meshes/link_016.stl scale=0.001 0.001 0.001
- added link link_017, mass 1.2954622871398063; collision mesh filename=package://robot_arm_description/meshes/link_017.stl scale=0.001 0.001 0.001; visual mesh filename=package://robot_arm_description/meshes/link_017.stl scale=0.001 0.001 0.001
- added link link_018, mass 0.01616774590367161; collision mesh filename=package://robot_arm_description/meshes/link_018.stl scale=0.001 0.001 0.001; visual mesh filename=package://robot_arm_description/meshes/link_018.stl scale=0.001 0.001 0.001
- added link link_019, mass 0.10912049174690079; collision mesh filename=package://robot_arm_description/meshes/link_019.stl scale=0.001 0.001 0.001; visual mesh filename=package://robot_arm_description/meshes/link_019.stl scale=0.001 0.001 0.001
- added link link_020, mass 0.020910021649792748; collision mesh filename=package://robot_arm_description/meshes/link_020.stl scale=0.001 0.001 0.001; visual mesh filename=package://robot_arm_description/meshes/link_020.stl scale=0.001 0.001 0.001
- added link link_021, mass 0.02091002164979277; collision mesh filename=package://robot_arm_description/meshes/link_021.stl scale=0.001 0.001 0.001; visual mesh filename=package://robot_arm_description/meshes/link_021.stl scale=0.001 0.001 0.001
- added link link_022, mass 0.024775801570545392; collision mesh filename=package://robot_arm_description/meshes/link_022.stl scale=0.001 0.001 0.001; visual mesh filename=package://robot_arm_description/meshes/link_022.stl scale=0.001 0.001 0.001
- added link link_023, mass 0.10879656543491555; collision mesh filename=package://robot_arm_description/meshes/link_023.stl scale=0.001 0.001 0.001; visual mesh filename=package://robot_arm_description/meshes/link_023.stl scale=0.001 0.001 0.001
- added link link_024, mass 0.03369324095260379; collision mesh filename=package://robot_arm_description/meshes/link_024.stl scale=0.001 0.001 0.001; visual mesh filename=package://robot_arm_description/meshes/link_024.stl scale=0.001 0.001 0.001
- added link link_025, mass 0.026632124946508604; collision mesh filename=package://robot_arm_description/meshes/link_025.stl scale=0.001 0.001 0.001; visual mesh filename=package://robot_arm_description/meshes/link_025.stl scale=0.001 0.001 0.001
- added link link_026, mass 0.03435402640600835; collision mesh filename=package://robot_arm_description/meshes/link_026.stl scale=0.001 0.001 0.001; visual mesh filename=package://robot_arm_description/meshes/link_026.stl scale=0.001 0.001 0.001
- added link link_027, mass 0.013742837703337476; collision mesh filename=package://robot_arm_description/meshes/link_027.stl scale=0.001 0.001 0.001; visual mesh filename=package://robot_arm_description/meshes/link_027.stl scale=0.001 0.001 0.001
- added link link_028, mass 0.12370727931856874; collision mesh filename=package://robot_arm_description/meshes/link_028.stl scale=0.001 0.001 0.001; visual mesh filename=package://robot_arm_description/meshes/link_028.stl scale=0.001 0.001 0.001
- added link link_029, mass 0.1091204917469009; collision mesh filename=package://robot_arm_description/meshes/link_029.stl scale=0.001 0.001 0.001; visual mesh filename=package://robot_arm_description/meshes/link_029.stl scale=0.001 0.001 0.001
- added link link_030, mass 0.0015707963267949652; collision mesh filename=package://robot_arm_description/meshes/link_030.stl scale=0.001 0.001 0.001; visual mesh filename=package://robot_arm_description/meshes/link_030.stl scale=0.001 0.001 0.001
- added link link_031, mass 0.45227624478140094; collision mesh filename=package://robot_arm_description/meshes/link_031.stl scale=0.001 0.001 0.001; visual mesh filename=package://robot_arm_description/meshes/link_031.stl scale=0.001 0.001 0.001
- added link link_032, mass 0.05007124655260372; collision mesh filename=package://robot_arm_description/meshes/link_032.stl scale=0.001 0.001 0.001; visual mesh filename=package://robot_arm_description/meshes/link_032.stl scale=0.001 0.001 0.001
- added link link_033, mass 0.024380202336228632; collision mesh filename=package://robot_arm_description/meshes/link_033.stl scale=0.001 0.001 0.001; visual mesh filename=package://robot_arm_description/meshes/link_033.stl scale=0.001 0.001 0.001
- added link link_034, mass 0.02073065249254581; collision mesh filename=package://robot_arm_description/meshes/link_034.stl scale=0.001 0.001 0.001; visual mesh filename=package://robot_arm_description/meshes/link_034.stl scale=0.001 0.001 0.001
- added link link_035, mass 0.01887089370282533; collision mesh filename=package://robot_arm_description/meshes/link_035.stl scale=0.001 0.001 0.001; visual mesh filename=package://robot_arm_description/meshes/link_035.stl scale=0.001 0.001 0.001
- added link link_036, mass 0.034085353103894385; collision mesh filename=package://robot_arm_description/meshes/link_036.stl scale=0.001 0.001 0.001; visual mesh filename=package://robot_arm_description/meshes/link_036.stl scale=0.001 0.001 0.001
- added link link_037, mass 0.031236901804661328; collision mesh filename=package://robot_arm_description/meshes/link_037.stl scale=0.001 0.001 0.001; visual mesh filename=package://robot_arm_description/meshes/link_037.stl scale=0.001 0.001 0.001
- added link link_038, mass 0.02374288789450661; collision mesh filename=package://robot_arm_description/meshes/link_038.stl scale=0.001 0.001 0.001; visual mesh filename=package://robot_arm_description/meshes/link_038.stl scale=0.001 0.001 0.001
- added link link_039, mass 0.31431191189124963; collision mesh filename=package://robot_arm_description/meshes/link_039.stl scale=0.001 0.001 0.001; visual mesh filename=package://robot_arm_description/meshes/link_039.stl scale=0.001 0.001 0.001
- added link link_040, mass 0.05689558566859283; collision mesh filename=package://robot_arm_description/meshes/link_040.stl scale=0.001 0.001 0.001; visual mesh filename=package://robot_arm_description/meshes/link_040.stl scale=0.001 0.001 0.001
- added link link_041, mass 0.09721724258742875; collision mesh filename=package://robot_arm_description/meshes/link_041.stl scale=0.001 0.001 0.001; visual mesh filename=package://robot_arm_description/meshes/link_041.stl scale=0.001 0.001 0.001
- added link link_042, mass 0.008257662906206078; collision mesh filename=package://robot_arm_description/meshes/link_042.stl scale=0.001 0.001 0.001; visual mesh filename=package://robot_arm_description/meshes/link_042.stl scale=0.001 0.001 0.001
- added link link_043, mass 0.008257662983629954; collision mesh filename=package://robot_arm_description/meshes/link_043.stl scale=0.001 0.001 0.001; visual mesh filename=package://robot_arm_description/meshes/link_043.stl scale=0.001 0.001 0.001
- added link link_044, mass 0.010975108826546717; collision mesh filename=package://robot_arm_description/meshes/link_044.stl scale=0.001 0.001 0.001; visual mesh filename=package://robot_arm_description/meshes/link_044.stl scale=0.001 0.001 0.001
- added link link_045, mass 0.010975108826539954; collision mesh filename=package://robot_arm_description/meshes/link_045.stl scale=0.001 0.001 0.001; visual mesh filename=package://robot_arm_description/meshes/link_045.stl scale=0.001 0.001 0.001
- added link link_046, mass 0.008257662906252378; collision mesh filename=package://robot_arm_description/meshes/link_046.stl scale=0.001 0.001 0.001; visual mesh filename=package://robot_arm_description/meshes/link_046.stl scale=0.001 0.001 0.001
- added link link_047, mass 0.008257662983629954; collision mesh filename=package://robot_arm_description/meshes/link_047.stl scale=0.001 0.001 0.001; visual mesh filename=package://robot_arm_description/meshes/link_047.stl scale=0.001 0.001 0.001
- added link link_048, mass 0.015261011971620197; collision mesh filename=package://robot_arm_description/meshes/link_048.stl scale=0.001 0.001 0.001; visual mesh filename=package://robot_arm_description/meshes/link_048.stl scale=0.001 0.001 0.001
- added link link_049, mass 0.07922324071673989; collision mesh filename=package://robot_arm_description/meshes/link_049.stl scale=0.001 0.001 0.001; visual mesh filename=package://robot_arm_description/meshes/link_049.stl scale=0.001 0.001 0.001
- added link link_050, mass 0.015261011971620171; collision mesh filename=package://robot_arm_description/meshes/link_050.stl scale=0.001 0.001 0.001; visual mesh filename=package://robot_arm_description/meshes/link_050.stl scale=0.001 0.001 0.001
- added link link_051, mass 0.06250206355985272; collision mesh filename=package://robot_arm_description/meshes/link_051.stl scale=0.001 0.001 0.001; visual mesh filename=package://robot_arm_description/meshes/link_051.stl scale=0.001 0.001 0.001
- added link link_052, mass 0.005422863209115555; collision mesh filename=package://robot_arm_description/meshes/link_052.stl scale=0.001 0.001 0.001; visual mesh filename=package://robot_arm_description/meshes/link_052.stl scale=0.001 0.001 0.001
- added link link_053, mass 0.012642489573939816; collision mesh filename=package://robot_arm_description/meshes/link_053.stl scale=0.001 0.001 0.001; visual mesh filename=package://robot_arm_description/meshes/link_053.stl scale=0.001 0.001 0.001
- added link link_054, mass 0.012642489573942336; collision mesh filename=package://robot_arm_description/meshes/link_054.stl scale=0.001 0.001 0.001; visual mesh filename=package://robot_arm_description/meshes/link_054.stl scale=0.001 0.001 0.001
- added link link_055, mass 0.00335380053643404; collision mesh filename=package://robot_arm_description/meshes/link_055.stl scale=0.001 0.001 0.001; visual mesh filename=package://robot_arm_description/meshes/link_055.stl scale=0.001 0.001 0.001
- added link link_056, mass 0.013998379225321508; collision mesh filename=package://robot_arm_description/meshes/link_056.stl scale=0.001 0.001 0.001; visual mesh filename=package://robot_arm_description/meshes/link_056.stl scale=0.001 0.001 0.001
- added link link_057, mass 0.013998377200492646; collision mesh filename=package://robot_arm_description/meshes/link_057.stl scale=0.001 0.001 0.001; visual mesh filename=package://robot_arm_description/meshes/link_057.stl scale=0.001 0.001 0.001
- link base_link: mass 0.7385873333015308 -> 0.1213729503132452
Joints:
- removed joint Revolute 23
- removed joint Revolute 29
- removed joint Revolute 42
- removed joint Revolute 48
- removed joint Revolute 72
- removed joint Rigid 20
- removed joint Rigid 21
- removed joint Rigid 22
- removed joint Rigid 24
- removed joint Rigid 25
- removed joint Rigid 26
- removed joint Rigid 27
- removed joint Rigid 28
- removed joint Rigid 30
- removed joint Rigid 31
- removed joint Rigid 32
- removed joint Rigid 33
- removed joint Rigid 34
- removed joint Rigid 35
- removed joint Rigid 36
- removed joint Rigid 37
- removed joint Rigid 38
- removed joint Rigid 39
- removed joint Rigid 40
- removed joint Rigid 43
- removed joint Rigid 44
- removed joint Rigid 45
- removed joint Rigid 46
- removed joint Rigid 47
- removed joint Rigid 49
- removed joint Rigid 50
- removed joint Rigid 51
- removed joint Rigid 52
- removed joint Rigid 62
- removed joint Rigid 63
- removed joint Rigid 64
- removed joint Rigid 65
- removed joint Rigid 66
- removed joint Rigid 71
- removed joint Rigid 73
- added joint arm_joint_1: type continuous, parent link_031, child link_028, origin xyz=0.0 0.0 0.04649999999999999 rpy=0.0 -0.0 0.0, axis 0.0 0.0 1.0, limit effort=10.6 velocity=3.14159265358979
- added joint arm_joint_2: type revolute, parent link_013, child link_015, origin xyz=0.0 0.0 -0.04650000000000001 rpy=0.0 -0.0 0.0, axis 0.0 -0.0 -1.0, limit lower=0 upper=3.14159265358979 effort=106 velocity=0.314159265358979
- added joint arm_joint_3: type revolute, parent link_017, child link_021, origin xyz=0.0 0.0 -0.07550000000000001 rpy=0.0 -0.0 0.0, axis 0.0 0.0 -1.0, limit lower=0 upper=3.14159265358979 effort=106 velocity=0.314159265358979
- added joint arm_joint_4: type revolute, parent link_006, child link_038, origin xyz=0.0 0.06337296 0.0 rpy=3.141592653589793 -0.0 3.141592653589793, axis 0.0 2.6716461825402365e-33 -1.0, limit lower=-0.610865238198015 upper=0.872664625997165 effort=10.6 velocity=3.14159265358979
- added joint arm_joint_5: type continuous, parent link_040, child link_033, origin xyz=-0.030999999999999996 0.0007499999999999929 0.003899999999999997 rpy=-1.3358230912699144e-33 -4.09841728479371e-34 0.0, axis 0.0 -1.3358230912699144e-33 1.0, limit effort=1.5 velocity=6.38790506229925
- added joint fixed_joint_001: type fixed, parent base_link, child link_029, origin xyz=0.0 0.01 0.004 rpy=0.0 -0.0 0.0
- added joint fixed_joint_002: type fixed, parent base_link, child link_031, origin xyz=0.0 0.01 0.004 rpy=0.0 -0.0 0.0
- added joint fixed_joint_003: type fixed, parent link_031, child link_030, origin xyz=0.0 0.0 0.04649999999999999 rpy=0.0 -0.0 0.0
- added joint fixed_joint_004: type fixed, parent link_028, child link_003, origin xyz=0.0 0.0 0.0040000000000000036 rpy=0.0 -0.0 7.1287974851291655e-62
- added joint fixed_joint_005: type fixed, parent link_028, child link_001, origin xyz=0.0 0.0 0.0040000000000000036 rpy=3.141592653589793 -0.0 7.1287974851291655e-62
- added joint fixed_joint_006: type fixed, parent link_003, child link_016, origin xyz=0.06215 -0.00045606 0.05999999999999999 rpy=-3.141592653589793 -1.5707963267948966 0
- added joint fixed_joint_007: type fixed, parent link_016, child link_014, origin xyz=0.0 -0.006000000000000001 -0.0675 rpy=0.0 -0.0 0.0
- added joint fixed_joint_008: type fixed, parent link_014, child link_013, origin xyz=0.0 0.0 -0.010299999999999998 rpy=0.0 -0.0 0.0
- added joint fixed_joint_009: type fixed, parent link_015, child link_012, origin xyz=0.0 0.0 -0.014800000000000004 rpy=0.0 -0.0 0.0
- added joint fixed_joint_010: type fixed, parent link_012, child link_002, origin xyz=-0.0009999999999999966 0.15 -0.001999999999999993 rpy=1.5707963267948966 -1.5707963267948966 0
- added joint fixed_joint_011: type fixed, parent link_002, child link_022, origin xyz=0.001999999999999993 -0.061 -0.143 rpy=1.5707963267948966 -0.0 -1.5707963267948966
- added joint fixed_joint_012: type fixed, parent link_002, child link_025, origin xyz=-0.002000000000000011 0.04699999999999999 -0.013818960000000012 rpy=-1.5707963267948966 -1.5707963267948966 0
- added joint fixed_joint_013: type fixed, parent link_012, child link_026, origin xyz=0.04900000000000002 0.13565161 -0.001999999999999993 rpy=1.5707963267948966 -1.5707963267948966 0
- added joint fixed_joint_014: type fixed, parent link_026, child link_010, origin xyz=0.1586 0.0 -0.025 rpy=0.0 -0.0 0.0
- added joint fixed_joint_015: type fixed, parent link_026, child link_011, origin xyz=0.1586 0.0 0.0 rpy=3.141592653589793 -0.0 0.0
- added joint fixed_joint_016: type fixed, parent link_011, child link_020, origin xyz=0.001999999999999993 -0.04900000000000002 -0.13565161 rpy=-1.5707963267948966 -0.0 1.5707963267948966
- added joint fixed_joint_017: type fixed, parent link_022, child link_019, origin xyz=0.0 0.0 -0.030300000000000004 rpy=0.0 -0.0 0.0
- added joint fixed_joint_018: type fixed, parent link_019, child link_018, origin xyz=0.0 0.0 -0.044000000000000004 rpy=0.0 -0.0 0.0
- added joint fixed_joint_019: type fixed, parent link_018, child link_017, origin xyz=0.0 0.0 -0.04070000000000001 rpy=0.0 -0.0 0.0
- added joint fixed_joint_020: type fixed, parent link_021, child link_004, origin xyz=0.0 0.0 0.016500000000000004 rpy=3.141592653589793 -0.0 0.0
- added joint fixed_joint_021: type fixed, parent link_004, child link_032, origin xyz=0.10800000000000001 -0.10673997 0.0 rpy=-1.5707963267948966 -0.0 -1.5707963267948966
- added joint fixed_joint_022: type fixed, parent link_004, child link_024, origin xyz=0.011999999999999993 -0.10673997 0.0 rpy=-1.5707963267948966 -0.0 1.5707963267948966
- added joint fixed_joint_023: type fixed, parent link_004, child link_008, origin xyz=0.06 -0.19462704 0.0 rpy=-1.5707963267948966 -0.0 0.0
- added joint fixed_joint_024: type fixed, parent link_008, child link_006, origin xyz=0.0 0.06865 0.0 rpy=-1.5707963267948966 5.473822126268817e-48 3.141592653589793
- added joint fixed_joint_025: type fixed, parent link_038, child link_023, origin xyz=0.0 0.0 0.003999999999999999 rpy=3.141592653589793 -0.0 0.0
- added joint fixed_joint_026: type fixed, parent link_038, child link_036, origin xyz=0.010500000000000008 0.0 -0.006600000000000002 rpy=0.0 -0.0 0.0
- added joint fixed_joint_027: type fixed, parent link_036, child link_035, origin xyz=0.0035000000000000144 0.094 -0.005 rpy=0.0 -0.0 0.0
- added joint fixed_joint_028: type fixed, parent link_036, child link_034, origin xyz=-0.013000000000000008 0.094 -0.005 rpy=0.0 -0.0 0.0
- added joint fixed_joint_029: type fixed, parent link_032, child link_005, origin xyz=0.0 0.1943 0.0 rpy=3.141592653589793 -0.0 -3.141592653589793
- added joint fixed_joint_030: type fixed, parent link_005, child link_009, origin xyz=-0.08788706999999998 0.0 0.04800000000000001 rpy=-3.141592653589793 -1.5707963267948966 0
- added joint fixed_joint_031: type fixed, parent link_009, child link_007, origin xyz=0.0 0.06865 0.0 rpy=-1.5707963267948966 5.473822126268817e-48 3.141592653589793
- added joint fixed_joint_032: type fixed, parent link_007, child link_027, origin xyz=0.0 0.06337296 0.0 rpy=3.141592653589793 -0.0 0.0
- added joint fixed_joint_033: type fixed, parent link_035, child link_037, origin xyz=0.0 0.0 0.08190000000000001 rpy=0.0 -0.0 0.0
- added joint fixed_joint_034: type fixed, parent link_036, child link_040, origin xyz=-0.004750000000000015 0.095 0.014950000000000001 rpy=-1.5707963267948966 1.5707963267948966 0
- added joint fixed_joint_035: type fixed, parent link_033, child link_039, origin xyz=0.0 0.0 0.005099999999999998 rpy=-3.141592653589793 1.1583765596690715e-32 -1.9721522630525295e-31
- added joint fixed_joint_036: type fixed, parent link_039, child link_041, origin xyz=0.0 0.0 -0.073 rpy=0.0 9.298773838736199e-33 0.0
- added joint fixed_joint_037: type fixed, parent link_041, child link_051, origin xyz=0.0 0.001999999999999993 -0.01 rpy=1.5707963267948966 -1.9721522630525295e-31 1.5707963267948966
- added joint fixed_joint_038: type fixed, parent link_055, child link_052, origin xyz=0.0 0.0 0.01 rpy=0.0 -0.0 0.0
- added joint fixed_joint_039: type fixed, parent link_056, child link_053, origin xyz=0.0 0.0 0.01 rpy=0.0 -0.0 -8.344469655179642e-31
- added joint fixed_joint_040: type fixed, parent link_057, child link_054, origin xyz=0.0 0.0 0.01 rpy=0.0 -9.860761315262648e-32 -5.551115123125708e-17
- added joint gripper_drive_joint: type revolute, parent link_051, child link_055, origin xyz=0.01800000000000001 -0.015071330000000015 -0.01110653 rpy=-3.141592653589793 -1.5707963267948966 0, axis 0.0 1.9721522630525295e-31 1.0, limit lower=-0.872664625997165 upper=1.0471975511966 effort=1.5 velocity=6.38790506229925
- added joint gripper_left_crank_joint: type revolute, parent link_049, child link_056, origin xyz=-0.03872177665071526 0.12873695533149415 2.2351752448912522e-10 rpy=2.848891993443736e-16 2.6206037754179146e-15 -1.570796326794897, axis 0.0 0.0 1.0, limit lower=-0.581776417331443 upper=0.698131700797732 effort=1.5 velocity=4.25860337486616, mimic joint=gripper_drive_joint multiplier=0.666666666666667 offset=0
- added joint gripper_left_finger_fixed: type fixed, parent link_046, child link_048, origin xyz=-0.02600885 0.035181150000000015 0.01 rpy=1.5707963267948966 4.794114453978405e-32 -3.138138633664991
- added joint gripper_left_inner_joint: type revolute, parent link_049, child link_044, origin xyz=-0.013843856650715232 0.13878695533149416 2.23517560016262e-10 rpy=-3.141592653589793 2.6206037754179146e-15 -1.570796326794897, axis 0.0 -0.0 1.0, limit lower=-0.698131700797732 upper=0.581776417331443 effort=1.5 velocity=4.25860337486616, mimic joint=gripper_drive_joint multiplier=-0.666666666666667 offset=0
- added joint gripper_left_lower_jaw_joint: type revolute, parent link_056, child link_042, origin xyz=0.05516076 0.04309629999999998 0.0 rpy=3.141592653589793 -0.0 -8.344469655179642e-31, axis 0.0 0.0 1.0, limit lower=-0.581776417331443 upper=0.698131700797732 effort=1.5 velocity=4.25860337486616, mimic joint=gripper_drive_joint multiplier=0.666666666666667 offset=0
- added joint gripper_left_upper_jaw_joint: type revolute, parent link_056, child link_046, origin xyz=0.05516076 0.04309629999999998 0.01 rpy=0.0 -0.0 -8.344469655179642e-31, axis 0.0 0.0 1.0, limit lower=-0.698131700797732 upper=0.581776417331443 effort=1.5 velocity=4.25860337486616, mimic joint=gripper_drive_joint multiplier=-0.666666666666667 offset=0
- added joint gripper_linkage_base_fixed: type fixed, parent link_051, child link_049, origin xyz=0.01799999977648284 -0.08282177665071525 0.14989347533149386 rpy=-1.570796326794898 5.5506916066521747e-17 -1.570796326794897
- added joint gripper_right_crank_joint: type revolute, parent link_049, child link_057, origin xyz=-0.03872177665071526 0.16483695533149423 2.2351763107053558e-10 rpy=2.848891993443736e-16 2.6206037754179146e-15 -1.570796326794897, axis 0.0 0.0 1.0, limit lower=-0.698131700797732 upper=0.581776417331443 effort=1.5 velocity=4.25860337486616, mimic joint=gripper_drive_joint multiplier=-0.666666666666667 offset=0
- added joint gripper_right_finger_fixed: type fixed, parent link_047, child link_050, origin xyz=0.026004009999999998 0.033762030000000005 0.009000000000000022 rpy=-1.5707963267948966 -1.4791053741944002e-31 3.138138633664991
- added joint gripper_right_inner_joint: type revolute, parent link_049, child link_045, origin xyz=-0.013843856650715232 0.1547869553314942 2.2351759554339879e-10 rpy=-3.141592653589793 2.6206037754179146e-15 -1.570796326794897, axis 0.0 -0.0 1.0, limit lower=-0.581776417331443 upper=0.698131700797732 effort=1.5 velocity=4.25860337486616, mimic joint=gripper_drive_joint multiplier=0.666666666666667 offset=0
- added joint gripper_right_lower_jaw_joint: type revolute, parent link_057, child link_043, origin xyz=-0.05516075 0.04309629999999998 0.0 rpy=3.141592653589793 -9.860761315262648e-32 -5.551115123125708e-17, axis -9.860761315262648e-32 -0.0 1.0, limit lower=-0.698131700797732 upper=0.581776417331443 effort=1.5 velocity=4.25860337486616, mimic joint=gripper_drive_joint multiplier=-0.666666666666667 offset=0
- added joint gripper_right_upper_jaw_joint: type revolute, parent link_057, child link_047, origin xyz=-0.05516075 0.04309629999999998 0.01 rpy=0.0 -9.860761315262648e-32 -5.551115123125708e-17, axis 9.860761315262648e-32 0.0 1.0, limit lower=-0.581776417331443 upper=0.698131700797732 effort=1.5 velocity=4.25860337486616, mimic joint=gripper_drive_joint multiplier=0.666666666666667 offset=0
