Commit message: feat(robot_arm_description): Isaac Sim export로 팔+그리퍼 URDF 전면 교체
RViz에서 팔 2/3축이 계속 이상하게 보이는 문제가 있었음. 원인을 진단해보니 기존
Fusion360 fusion2urdf 계열(VerNOmiddle) export의 joint_2 축 부호가 실제와
반대였고, 그 아래 매달린 3축 이하가 덩달아 이상해 보인 것이었음. 사용자가 이
CAD 파이프라인 자체를 신뢰하기 어렵다고 판단해, Isaac Sim에서 새로 뽑은
robotarm_urdf_20260711.urdf(+closed_loop.usd)로 URDF를 통째로 교체하기로 결정.

- mesh 58개: 원본에 딸린 meshes_ascii STL이 실제로는 어디에도 없어서(Isaac Sim
  exporter가 geometry를 USD에만 남김), usd-core(pxr)로 USD 안의 raw mesh point를
  직접 추출 → numpy-stl로 binary STL 변환 → robot_arm_description/meshes/ 전체
  교체(기존 56개 mesh, gripper_a 서브트리 포함 전량 대체).
- 그리퍼가 이제 실제 구동 조인트 gripper_drive_joint 하나 + URDF <mimic> 태그로
  종속되는 8개(크랭크/조 관절)로 정식 표현됨 — 기존엔 평행 4절링크의 닫힌 루프를
  중복 링크를 잘라내는 방식으로 근사해 실제 기구 구속을 못 담았음.
- 조인트 이름 체계 변경(joint_1~5, gripper_a_joint5/6 → arm_joint_1~5,
  gripper_drive_joint)을 dynamixel_control(moveit_dynamixel_bridge.py의
  JOINT_CONFIG, arm_fsm_node.py의 ARM_JOINT_NAMES/tip_link 기본값,
  gripper_presets.py의 gripper_joints)과 robot_arm_moveit_config 전체(SRDF
  chain/group/group_state/end_effector/disable_collisions, joint_limits.yaml,
  initial_positions.yaml, moveit_controllers.yaml, ros2_controllers.yaml,
  robot_arm.ros2_control.xacro)에 걸쳐 갱신.
- SRDF disable_collisions는 새 58-link 토폴로지의 Adjacent(부모-자식) 쌍만
  URDF에서 프로그램적으로 자동 도출해 채움 — 기어 치합 등 자세무관 Default 쌍은
  실제 충돌체크 없이 지어내지 않고 비워둠(MoveIt Setup Assistant 재실행 필요,
  주석으로 명시).
- 레거시 dynamixel_position_node.py(별도 P-control 파이프라인, joint_1~3 이름
  그대로)는 범위 밖으로 판단해 의도적으로 안 건드림.

컨테이너에서 colcon build + display.launch.py로 전체 링크 로드, mimic 조인트
자동 종속 확인, 사용자가 RViz 육안으로도 확인 완료.

Co-Authored-By: Claude Sonnet 5 <noreply@anthropic.com>

File: ros2_ws/src/robot_arm_description/urdf/robot_arm.urdf.xacro (robot description, xacro)
@@ -1,20 +1,13 @@
 <?xml version="1.0"?>
-<!-- 그리퍼 모듈화 메인 xacro: 몸체(robot_arm.urdf) + 그리퍼(urdf/grippers/*.xacro)를 조립.
-     그리퍼 모듈화 가이드(§4)의 sirumi.urdf.xacro 패턴을 그대로 적용.
-     robot_arm.urdf는 <robot> 태그를 가진 완성 URDF지만, xacro:include는 루트 태그 이름과
-     무관하게 자식 엘리먼트를 그대로 이 파일의 <robot>에 이어붙이므로 별도 body-only 파일 없이 재사용 가능.
-     wrist_to_gripper 조인트의 origin/rpy는 CAD팀이 제공한 위치 확정용 통합 export
-     (2026_07_10_Arm_with_Gripper_Ver2, Gripper_1 단일메쉬)의 Rigid 74 조인트(module_connector
-     기준 xyz=0,-0.073,0)를 gripper_a_base_link.stl과의 Kabsch 강체정합(양쪽 메쉬가 동일 부품임을
-     삼각형수 일치로 확인, 정합 오차 ~8um)으로 역산한 값 — 이전엔 rpy=0으로 두는 실수가 있었는데
-     실제로는 -90°(Z) 회전이 필요해서 그리퍼가 팔 진행방향이 아니라 옆으로 삐져나와 보이는 원인이었음. -->
+<!-- 메인 xacro: robot_arm.urdf(2026-07-15 VerNOmiddle 통합 재export 기준, 팔+gripper_a 전체가
+     이미 하나의 tree)를 그대로 include. robot_arm.urdf는 <robot> 태그를 가진 완성 URDF지만,
+     xacro:include는 루트 태그 이름과 무관하게 자식 엘리먼트를 그대로 이 파일의 <robot>에 이어붙임.
+     이전엔 여기서 xacro:arg gripper로 그리퍼 모듈(urdf/grippers/*.xacro)을 골라 wrist_to_gripper
+     fixed joint로 짜맞췄으나, 서로 다른 CAD export(팔/그리퍼 각각 다른 리비전)의 좌표계를 맞추는
+     시도가 반복적으로 어긋나 폐기(2026-07-15, 사용자 결정) — robot_arm.urdf 헤더 주석 참고.
+     그리퍼 "모듈화"는 이제 로직 레벨(dynamixel_control의 gripper_type/gripper_presets.py)에서만
+     유지되고, URDF 레벨 스왑은 없음. 그리퍼를 실제로 교체하려면 robot_arm.urdf 자체를 새 통합
+     export로 다시 만들어야 함(urdf/grippers/ 디렉토리는 더 이상 사용 안 함). -->
 <robot name="robot_arm" xmlns:xacro="http://www.ros.org/wiki/xacro">
-  <xacro:arg name="gripper" default="gripper_a"/>
   <xacro:include filename="$(find robot_arm_description)/urdf/robot_arm.urdf"/>
-  <xacro:include filename="$(find robot_arm_description)/urdf/grippers/$(arg gripper).xacro"/>
-  <joint name="wrist_to_gripper" type="fixed">
-    <origin xyz="-0.146787 -0.166071 0.02" rpy="0 0 -1.5707963"/>
-    <parent link="module_connector_5axis_Component41_1"/>
-    <child link="$(arg gripper)_base_link"/>
-  </joint>
 </robot>

File: ros2_ws/src/robot_arm_moveit_config/config/robot_arm.ros2_control.xacro (robot description, xacro)
@@ -8,50 +8,43 @@
                 <plugin>mock_components/GenericSystem</plugin>
             </hardware>
-            <joint name="Revolute 23">
+            <joint name="arm_joint_1">
                 <command_interface name="position"/>
                 <state_interface name="position">
-                  <param name="initial_value">${initial_positions['Revolute 23']}</param>
+                  <param name="initial_value">${initial_positions['arm_joint_1']}</param>
                 </state_interface>
                 <state_interface name="velocity"/>
             </joint>
-            <joint name="Revolute 29">
+            <joint name="arm_joint_2">
                 <command_interface name="position"/>
                 <state_interface name="position">
-                  <param name="initial_value">${initial_positions['Revolute 29']}</param>
+                  <param name="initial_value">${initial_positions['arm_joint_2']}</param>
                 </state_interface>
                 <state_interface name="velocity"/>
             </joint>
-            <joint name="Revolute 42">
+            <joint name="arm_joint_3">
                 <command_interface name="position"/>
                 <state_interface name="position">
-                  <param name="initial_value">${initial_positions['Revolute 42']}</param>
+                  <param name="initial_value">${initial_positions['arm_joint_3']}</param>
                 </state_interface>
                 <state_interface name="velocity"/>
             </joint>
-            <joint name="Revolute 48">
+            <joint name="arm_joint_4">
                 <command_interface name="position"/>
                 <state_interface name="position">
-                  <param name="initial_value">${initial_positions['Revolute 48']}</param>
+                  <param name="initial_value">${initial_positions['arm_joint_4']}</param>
                 </state_interface>
                 <state_interface name="velocity"/>
             </joint>
-            <joint name="Revolute 72">
+            <joint name="arm_joint_5">
                 <command_interface name="position"/>
                 <state_interface name="position">
-                  <param name="initial_value">${initial_positions['Revolute 72']}</param>
+                  <param name="initial_value">${initial_positions['arm_joint_5']}</param>
                 </state_interface>
                 <state_interface name="velocity"/>
             </joint>
-            <joint name="gripper_a_joint5">
+            <joint name="gripper_drive_joint">
                 <command_interface name="position"/>
                 <state_interface name="position">
-                  <param name="initial_value">${initial_positions['gripper_a_joint5']}</param>
-                </state_interface>
-                <state_interface name="velocity"/>
-            </joint>
-            <joint name="gripper_a_joint6">
-                <command_interface name="position"/>
-                <state_interface name="position">
-                  <param name="initial_value">${initial_positions['gripper_a_joint6']}</param>
+                  <param name="initial_value">${initial_positions['gripper_drive_joint']}</param>
                 </state_interface>
                 <state_interface name="velocity"/>
