Commit message: Merge main into new

File: ros2_ws/src/robot_arm_moveit_config/config/robot_arm.urdf.xacro (robot description, xacro)
@@ -2,7 +2,11 @@
 <robot xmlns:xacro="http://www.ros.org/wiki/xacro" name="robot_arm">
     <xacro:arg name="initial_positions_file" default="initial_positions.yaml" />
-    <!-- Import robot_arm urdf file -->
     <xacro:include filename="$(find robot_arm_description)/urdf/robot_arm.urdf" />
-    <!-- Import control_xacro -->
+    <xacro:include filename="$(find robot_arm_description)/urdf/gripper_prefixed.xacro" />
+    <joint name="gripper_mount_joint" type="fixed">
+      <parent link="마지막_링크_이름"/>
+      <child link="gripper_base_link"/>
+      <origin xyz="0 0 0" rpy="0 0 0"/>
+    </joint>
     <xacro:include filename="robot_arm.ros2_control.xacro" />
     <xacro:robot_arm_ros2_control name="FakeSystem" initial_positions_file="$(arg initial_positions_file)"/>
