Commit message: fix(robot_arm_description): gripper_a 조인트 타입 수정 및 wrist_to_gripper 오프셋 재계산
- gripper_a.xacro: joint5/6를 continuous→revolute(±90도 limit)로 변경, link2/4·joint23에
  mimic 태그 복원(평행 4절링크 커플링 시각화 복구), <robot> 루트 태그 래퍼 추가
- robot_arm.urdf.xacro: wrist_to_gripper origin/rpy를 CAD 통합 export 기준 Kabsch 강체정합
  값으로 재계산(기존 rpy=0 오류로 그리퍼가 옆으로 삐져나오던 문제 수정)
- robot_arm_moveit_config: 위 변경 반영해 SRDF/controllers/joint_limits/initial_positions/
  ros2_control.xacro를 MoveIt Setup Assistant로 재생성

Co-Authored-By: Claude Sonnet 5 <noreply@anthropic.com>

File: ros2_ws/src/robot_arm_description/urdf/grippers/gripper_a.xacro (robot description, xacro)
@@ -330,16 +330,23 @@
   </collision>
 </link>
-<joint name="gripper_a_joint5" type="continuous">
+<!-- 실측 기구 개폐range/방향 미확정 placeholder, 사용자 수동 캘리브레이션 진행 중.
+     mimic(joint5<->joint6) 임시 해제 — 두 핑거 각도가 대칭이 아니라 -1 배율로는 안 맞음, 개별 지시로 재조정 예정.
+     range는 우선 넉넉하게(±1.5708rad=±90도) 잡아둠. -->
+<joint name="gripper_a_joint5" type="revolute">
   <origin xyz="0.01335 0.01805 0.036" rpy="0 0 0" />
   <parent link="gripper_a_top_plate" />
   <child link="gripper_a_link1" />
   <axis xyz="-0.0 0.0 -1.0" />
-</joint>
-<joint name="gripper_a_joint6" type="continuous">
+  <limit lower="-1.5708" upper="1.5708" effort="5" velocity="1.0" />
+</joint>
+<joint name="gripper_a_joint6" type="revolute">
   <origin xyz="0.01335 -0.01805 0.036" rpy="0 0 0" />
   <parent link="gripper_a_top_plate" />
   <child link="gripper_a_link3" />
   <axis xyz="-0.0 0.0 -1.0" />
-</joint>
+  <limit lower="-1.5708" upper="1.5708" effort="5" velocity="1.0" />
+</joint>
+<!-- link2는 평행4절링크의 두번째 크랭크 — link1(joint5)과 top_plate 기준 같은 각도로 돌아야 평행 유지됨.
+     루프 단순화로 독립 관절이 되며 구동과 무관하게 정지해 있던 것을 mimic으로 복원(같은 축·동일 부호). -->
 <joint name="gripper_a_joint7" type="continuous">
   <origin xyz="0.038228 0.008 0.036" rpy="0 0 0" />
@@ -347,5 +354,7 @@
   <child link="gripper_a_link2" />
   <axis xyz="-0.0 0.0 -1.0" />
-</joint>
+  <mimic joint="gripper_a_joint5" multiplier="1" offset="0" />
+</joint>
+<!-- link4 = link2와 대칭인 반대쪽 평행4절링크 크랭크, link3(joint6)를 따라감. -->
 <joint name="gripper_a_joint8" type="continuous">
   <origin xyz="0.038228 -0.008 0.036" rpy="0 0 0" />
@@ -353,4 +362,5 @@
   <child link="gripper_a_link4" />
   <axis xyz="-0.0 0.0 -1.0" />
+  <mimic joint="gripper_a_joint6" multiplier="1" offset="0" />
 </joint>
 <joint name="gripper_a_joint9" type="continuous">
@@ -400,4 +410,6 @@
   <axis xyz="-0.0 0.0 -1.0" />
 </joint>
+<!-- 24T(모터) - 36T(joint5측 gripper_a_link1) 직결 치합 기어비 24:36 = 2:3 → 모터가 그리퍼(joint5)의
+     2/3만큼 회전. 외접기어 치합이라 joint5/joint23 axis가 둘 다 base_link 기준 동일 -Z라 부호는 반대. -->
 <joint name="gripper_a_joint23" type="continuous">
   <origin xyz="0.0 0.0 0.01" rpy="0 0 0" />
@@ -405,4 +417,5 @@
   <child link="gripper_a_Spur_Gear_24_teeth__2__1" />
   <axis xyz="0.0 -0.0 -1.0" />
+  <mimic joint="gripper_a_joint5" multiplier="-0.66667" offset="0" />
 </joint>
 <joint name="gripper_a_fixed24" type="fixed">

File: ros2_ws/src/robot_arm_description/urdf/robot_arm.urdf.xacro (robot description, xacro)
@@ -4,6 +4,9 @@
      robot_arm.urdf는 <robot> 태그를 가진 완성 URDF지만, xacro:include는 루트 태그 이름과
      무관하게 자식 엘리먼트를 그대로 이 파일의 <robot>에 이어붙이므로 별도 body-only 파일 없이 재사용 가능.
-     wrist_to_gripper 조인트의 origin은 module_connector_5axis_Component41_1(팔 끝단) 원점 기준
-     실측 마운트 위치(x=147.544mm, y=0, z=239.50mm, base_link 기준)에서 역산한 값 — CAD 실측 재확인 필요. -->
+     wrist_to_gripper 조인트의 origin/rpy는 CAD팀이 제공한 위치 확정용 통합 export
+     (2026_07_10_Arm_with_Gripper_Ver2, Gripper_1 단일메쉬)의 Rigid 74 조인트(module_connector
+     기준 xyz=0,-0.073,0)를 gripper_a_base_link.stl과의 Kabsch 강체정합(양쪽 메쉬가 동일 부품임을
+     삼각형수 일치로 확인, 정합 오차 ~8um)으로 역산한 값 — 이전엔 rpy=0으로 두는 실수가 있었는데
+     실제로는 -90°(Z) 회전이 필요해서 그리퍼가 팔 진행방향이 아니라 옆으로 삐져나와 보이는 원인이었음. -->
 <robot name="robot_arm" xmlns:xacro="http://www.ros.org/wiki/xacro">
   <xacro:arg name="gripper" default="gripper_a"/>
@@ -11,5 +14,5 @@
   <xacro:include filename="$(find robot_arm_description)/urdf/grippers/$(arg gripper).xacro"/>
   <joint name="wrist_to_gripper" type="fixed">
-    <origin xyz="0.136594 0.074544 0.0" rpy="0 0 0"/>
+    <origin xyz="-0.146787 -0.166071 0.02" rpy="0 0 -1.5707963"/>
     <parent link="module_connector_5axis_Component41_1"/>
     <child link="$(arg gripper)_base_link"/>

File: ros2_ws/src/robot_arm_moveit_config/config/robot_arm.ros2_control.xacro (robot description, xacro)
@@ -8,22 +8,50 @@
                 <plugin>mock_components/GenericSystem</plugin>
             </hardware>
-            <joint name="joint_1">
+            <joint name="Revolute 23">
                 <command_interface name="position"/>
                 <state_interface name="position">
-                  <param name="initial_value">${initial_positions['joint_1']}</param>
+                  <param name="initial_value">${initial_positions['Revolute 23']}</param>
                 </state_interface>
                 <state_interface name="velocity"/>
             </joint>
-            <joint name="joint_2">
+            <joint name="Revolute 29">
                 <command_interface name="position"/>
                 <state_interface name="position">
-                  <param name="initial_value">${initial_positions['joint_2']}</param>
+                  <param name="initial_value">${initial_positions['Revolute 29']}</param>
                 </state_interface>
                 <state_interface name="velocity"/>
             </joint>
-            <joint name="joint_3">
+            <joint name="Revolute 42">
                 <command_interface name="position"/>
                 <state_interface name="position">
-                  <param name="initial_value">${initial_positions['joint_3']}</param>
+                  <param name="initial_value">${initial_positions['Revolute 42']}</param>
+                </state_interface>
+                <state_interface name="velocity"/>
+            </joint>
+            <joint name="Revolute 48">
+                <command_interface name="position"/>
+                <state_interface name="position">
+                  <param name="initial_value">${initial_positions['Revolute 48']}</param>
+                </state_interface>
+                <state_interface name="velocity"/>
+            </joint>
+            <joint name="Revolute 72">
+                <command_interface name="position"/>
+                <state_interface name="position">
+                  <param name="initial_value">${initial_positions['Revolute 72']}</param>
+                </state_interface>
+                <state_interface name="velocity"/>
+            </joint>
+            <joint name="gripper_a_joint5">
+                <command_interface name="position"/>
+                <state_interface name="position">
+                  <param name="initial_value">${initial_positions['gripper_a_joint5']}</param>
+                </state_interface>
+                <state_interface name="velocity"/>
+            </joint>
+            <joint name="gripper_a_joint6">
+                <command_interface name="position"/>
+                <state_interface name="position">
+                  <param name="initial_value">${initial_positions['gripper_a_joint6']}</param>
                 </state_interface>
                 <state_interface name="velocity"/>

File: ros2_ws/src/robot_arm_moveit_config/config/robot_arm.urdf.xacro (robot description, xacro)
@@ -2,6 +2,6 @@
 <robot xmlns:xacro="http://www.ros.org/wiki/xacro" name="robot_arm">
     <xacro:arg name="initial_positions_file" default="initial_positions.yaml" />
-    <!-- Import robot_arm urdf file -->
-    <xacro:include filename="$(find robot_arm_description)/urdf/robot_arm.urdf" />
+    <!-- Import robot_arm urdf file (몸체 + gripper_a, robot_arm_description의 그리퍼 모듈화 xacro) -->
+    <xacro:include filename="$(find robot_arm_description)/urdf/robot_arm.urdf.xacro" />
     <!-- Import control_xacro -->
     <xacro:include filename="robot_arm.ros2_control.xacro" />
